Commit message: translated and working by bits

File: urdf/myrobot.gazebo.xacro (robot description, xacro)
@@ -1,4 +1,4 @@
 <?xml version="1.0"?>
-<robot name="myrobot_sim" xmlns:xacro="http://ros.org/wiki/xacro">
+<robot name="myrobot" xmlns:xacro="http://ros.org/wiki/xacro">
   <gazebo reference="cube_base">
   </gazebo>
@@ -11,4 +11,5 @@
     <maxVel>0.1</maxVel>
     <fdir1>1 0 0</fdir1>
+    <material>Gazebo/FlatBlack</material>
   </gazebo>
   <gazebo reference="wheel_right_link">
@@ -20,6 +21,7 @@
     <maxVel>0.1</maxVel>
     <fdir1>1 0 0</fdir1>
-  </gazebo>
-  <!-- <gazebo reference="RealSense">
+    <material>Gazebo/FlatBlack</material>
+  </gazebo>
+  <gazebo reference="RealSense">
     <sensor name="camera" type="depth">
       <update_rate>20</update_rate>
@@ -29,5 +31,5 @@
           <width>640</width>
           <height>480</height>
-          <format>R8G8B8</format>
+          <format>R8G8B8</format><!---->
         </image>
         <clip>
@@ -96,10 +98,12 @@
       </ray>
     </sensor>
-  </gazebo> -->
+  </gazebo>
 <!-- PLUGINS -->
-  <!-- <gazebo>
+  <gazebo>
     <plugin name="camera_plugin" filename="libdepth_camera_plugin.so">
       <baseline>0.2</baseline>
       <alwaysOn>true</alwaysOn>
+       <!-- Keep this zero, update_rate in the parent <sensor> tag
+        will control the frame rate. -->
       <updateRate>0.0</updateRate>
       <cameraName>camera_ir</cameraName>
@@ -123,6 +127,7 @@
       <hackBaseline>0</hackBaseline>
     </plugin>
-  </gazebo> -->
-  <!-- <gazebo>
+  </gazebo>
+  <gazebo>
+    <!-- Contact sensor plugin -->
     <plugin name="gazebo_ros_bumper_controller" filename="libcontact_plugin.so">
       <alwaysOn>true</alwaysOn>
@@ -130,7 +135,8 @@
       <bumperTopicName>/force/rightfront_sensor</bumperTopicName>
       <frameName>rightfront_force_sensor</frameName>
-    </plugin>
-  </gazebo>
-  <gazebo>
+    </plugin> <!-- -->
+  </gazebo>
+  <gazebo>
+  <!-- Contact sensor plugin -->
     <plugin name="gazebo_ros_bumper_controller" filename="libcontact_plugin.so">
       <alwaysOn>true</alwaysOn>
@@ -138,7 +144,8 @@
       <bumperTopicName>/force/leftfront_sensor</bumperTopicName>
       <frameName>leftfront_force_sensor</frameName>
-    </plugin>
-  </gazebo> -->
-  <!-- <gazebo>
+    </plugin> <!-- -->
+  </gazebo>
+  <gazebo>
+      <!-- Light sensor plugin -->
     <plugin name="myrobot" filename="liblight_sensor_plugin.so">
       <cameraName>camera2</cameraName>
@@ -160,12 +167,13 @@
       <pointCloudCutoff>0.4</pointCloudCutoff>
       <robotNamespace>/</robotNamespace>
-    </plugin>
-  </gazebo> -->
-  <!-- <gazebo>
+    </plugin> <!-- -->
+  </gazebo>
+  <gazebo>
+        <!-- Laser sensor plugin -->
     <plugin name="gazebo_ros_lds_lfcd_controller" filename="libgazebo_ros_laser.so">
       <topicName>scan</topicName>
       <frameName>cube_base</frameName>
     </plugin>
-  </gazebo> -->
+  </gazebo>
   <gazebo>
     <plugin name="cube_moving_code" filename="libdiff_drive_plugin.so">

File: urdf/myrobot.urdf.xacro (robot description, xacro)
@@ -26,15 +26,10 @@
         </geometry>
       </collision>
-     <visual name="visual">
-        <geometry>
-          <box size="0.19 0.134 0.047"/>
-        </geometry>
-      </visual>
-      <!-- <visual>
+      <visual>
         <origin xyz="0.02 0 -0.01" rpy="1.5707 0 1.5707"/>
         <geometry>
-          <mesh filename="package://myrobot/models/myroboturdf/meshes/Devastator.dae"/>
-        </geometry>
-      </visual> -->
+          <mesh filename="package://myrobot/models/myroboturdf/meshes/Devastator.dae" scale="1 1 1"/>
+        </geometry>
+      </visual>
       <collision name = "caster_collision">
       <origin xyz="-0.05 0 -0.03" rpy="0 0 0"/>
@@ -53,10 +48,4 @@
         </surface>
       </collision>
-      <visual name="caster_collision">
-      <origin xyz="-0.05 0 -0.03" rpy="0 0 0"/>
-        <geometry>
-          <sphere radius="0.05"/>
-        </geometry>
-      </visual>
       <collision name = 'caster_collision2'>
       <origin xyz="0.05 0 -0.03" rpy="0 0 0"/>
@@ -75,10 +64,4 @@
         </surface>
       </collision>
-      <visual name="caster_collision2">
-      <origin xyz="0.05 0 -0.03" rpy="0 0 0"/>
-        <geometry>
-          <sphere radius="0.05"/>
-        </geometry>
-      </visual>
     </link>
     <joint name="wheel_left_joint" type="continuous">
@@ -94,4 +77,5 @@
         <inertia ixx="0.00052666666" ixy="0" ixz="0" iyy="0.00052666666" iyz="0" izz="0.001"/>
       </inertial>
+      <!-- <pose>0. 0.087 0.06825 0 1.5707 1.5707 </pose> -->
       <collision>
         <origin xyz="0 0 0" rpy="0 0 0"/>
@@ -106,12 +90,27 @@
         </geometry>
       </visual>
+        <!--<visual name='visual'>
+          <geometry>
+            <cylinder>
+              <radius>.06825</radius>
+              <length>0.04</length>
+            </cylinder>
+          </geometry>
+          <material>
+            <ambient>0.1 0.1 0.1 1</ambient>
+            <diffuse>0.1 0.1 0.2 1</diffuse>
+            <specular>0 0 0 0</specular>
+            <emissive>0 0 0 1</emissive>
+          </material>
+        </visual> -->
     </link>
     <joint name="wheel_right_joint" type="continuous">
       <parent link="cube_base"/>
       <child link="wheel_right_link"/>
-      <origin xyz="0. -0.087 0.06825" rpy="0 0 0"/>
+      <origin xyz="0. -0.087 0.06825" rpy="0 1.5707 1.5707"/>
       <axis xyz="0 0 1"/>
     </joint>
-    <link name="wheel_right_link">
+    <link name="wheel_right_joint">
+      <!-- <pose>0. -0.087 0.06825 0 1.5707 1.5707 </pose> -->
       <inertial>
         <mass value="0.2"/>
@@ -119,4 +118,5 @@
         <inertia ixx="0.00052666666" ixy="0" ixz="0" iyy="0.00052666666" iyz="0" izz="0.001"/>
       </inertial>
+      <!-- <pose>0. 0.087 0.06825 0 1.5707 1.5707 </pose> -->
       <collision>
         <origin xyz="0 0 0" rpy="0 0 0"/>
@@ -132,9 +132,10 @@
       </visual>
     </link>
-    <!-- <joint name="BaseBoards_joint" type="fixed">
+    <joint name="BaseBoards_joint" type="fixed">
       <parent link="cube_base"/>
       <child link="BaseBoards"/>
       <origin xyz="-0.01 0 0.1435" rpy="0 0 0"/>
     </joint>
+    <!--%%%%%%%%%%%%%%%%%%%%%%%%%%%%%%%%%%%%%%%%%SUPPORTS%%%%%%%%%%%%%%%%%%%%%%%%%%%%%%%%%%%%%%%%%%%%%%-->
     <link name="BaseBoards">
       <inertial>
@@ -155,5 +156,17 @@
         </geometry>
       </visual>
-      <collision name = "stick1_collision">
+      <!-- <visual name="visual">
+        <pose>0.05 0 0 0 0 1.5707</pose>
+        <geometry>
+          <mesh><uri>model://myrobot/meshes/Supports/BaseBoards.dae</uri></mesh>
+        </geometry>
+        <material>
+          <ambient>0 0 0.196 0.490</ambient>
+          <diffuse>0.043 0.043 0.043 1</diffuse>
+          <specular>.027 .027 .459 64</specular>
+          <emissive>0.047 0.035 0.286 1</emissive>
+        </material>
+      </visual> -->
+      <!-- <collision name = "stick1_collision">
       <origin xyz="0.075 0.05 -0.02 " rpy="0 0 0"/>
         <geometry>
@@ -202,8 +215,7 @@
           <cylinder length="0.04" radius="0.002"/>
         </geometry>
-      </visual>
-    </link>
-     -->
-    <!-- <joint name="piastra_anteriore_joint" type="fixed">
+      </visual> -->
+    </link>
+    <joint name="piastra_anteriore_joint" type="fixed">
       <parent link="BaseBoards"/>
       <child link="piastra_anteriore"/>
@@ -228,6 +240,6 @@
         </geometry>
       </visual>
-    </link> -->
-    <!-- <joint name="supporto_sg90_joint" type="fixed">
+    </link>
+    <joint name="supporto_sg90_joint" type="fixed">
       <parent link="piastra_anteriore"/>
       <child link="supporto_sg90"/>
@@ -253,6 +265,5 @@
       </visual>
     </link>
-     -->
-    <!-- <joint name="supporto_piastra_albero_joint" type="fixed">
+    <joint name="supporto_piastra_albero_joint" type="fixed">
       <parent link="sg90h_shaft"/>
       <child link="supporto_piastra_albero"/>
@@ -277,6 +288,8 @@
         </geometry>
       </visual>
-    </link> -->
-    <!-- <joint name="supporto_pitch_servo_1_joint" type="fixed">
+      <!-- <pose>0.106 0.0005 0.109 0 0 0</pose> -->
+      <!--<pose>0 0 0 0 0 0</pose>-->
+    </link>
+    <joint name="supporto_pitch_servo_1_joint" type="fixed">
       <parent link="supporto_piastra_albero"/>
       <child link="supporto_pitch_servo_1"/>
@@ -285,4 +298,5 @@
     <gazebo>
     <link name='supporto_pitch_servo_1'>
+      <!-- <pose>0.106 0.038 0.114 0 0 4.71238</pose> -->
       <inertial>
         <mass>0.1</mass>
@@ -345,6 +359,6 @@
       </collision>
     </link>
-    </gazebo> -->
-    <!-- <joint name="supporto_pitch_servo_2_joint" type="fixed">
+    </gazebo>
+    <joint name="supporto_pitch_servo_2_joint" type="fixed">
       <parent link="supporto_pitch_servo_1"/>
       <child link="supporto_pitch_servo_2"/>
@@ -391,6 +405,6 @@
       </collision>
     </link>
-    </gazebo> -->
-    <!-- <joint name="supporto_pitch_servo_2_noservo_joint" type="fixed">
+    </gazebo>
+    <joint name="supporto_pitch_servo_2_noservo_joint" type="fixed">
       <parent link="supporto_pitch_servo_1"/>
       <child link="supporto_pitch_servo_2_noservo"/>
@@ -399,4 +413,6 @@
     <gazebo>
     <link name='supporto_pitch_servo_2_noservo'>
+    <!-- <self_collide>true</self_collide> -->
+      <!-- <pose>0.106 -0.056 0.116 0 0 1.5707</pose> -->
       <inertial>
         <mass>0.1</mass>
@@ -427,4 +443,18 @@
         </material>
       </visual>
+      <!-- <visual name='visual'>
+      <pose>0 0 0 0 0 0 </pose>
+        <geometry>
+          <box>
+            <size>0.0075 0.035 0.002</size>
+          </box>
+        </geometry>
+        <material>
+          <script>
+            <uri>file://media/materials/scripts/gazebo.material</uri>
+            <name>Gazebo/RedTransparent</name>
+          </script>
+        </material>
+      </visual> -->
       <collision name='collision_vertical'>
       <pose>-0.002375 0 0.018 0 0 0 </pose>
@@ -435,7 +465,21 @@
         </geometry>
       </collision>
-    </link>
-    </gazebo> -->
-    <!-- <joint name="supp_RS_joint" type="fixed">
+      <!-- <visual name='collision_vertical'>
+      <pose>-0.002375 0 0.018 0 0 0 </pose>
+        <geometry>
+          <box>
+            <size>0.002 0.019 0.036</size>
+          </box>
+        </geometry>
+        <material>
+          <script>
+            <uri>file://media/materials/scripts/gazebo.material</uri>
+            <name>Gazebo/RedTransparent</name>
+          </script>
+        </material>
+      </visual> -->
+    </link>
+    </gazebo>
+    <joint name="supp_RS_joint" type="fixed">
       <parent link="sg90v_shaft"/>
       <child link="supp_RS"/>
@@ -480,6 +524,7 @@
       </collision>
     </link>
-    </gazebo> -->
-    <!-- <joint name="RealSense_joint" type="fixed">
+    </gazebo>
+    <!--%%%%%%%%%%%%%%%%%%%%%%%%%%%%%%%%%%%%%%%%%SENSORS%%%%%%%%%%%%%%%%%%%%%%%%%%%%%%%%%%%%%%%%%%%%%%-->
+    <joint name="RealSense_joint" type="fixed">
       <parent link="supp_RS"/>
       <child link="RealSense"/>
@@ -498,6 +543,6 @@
           </geometry>
         </visual>
-    </link> -->
-    <!-- <joint name="rightfront_force_sensor_joint" type="fixed">
+    </link>
+    <joint name="rightfront_force_sensor_joint" type="fixed">
       <parent link="cube_base"/>
       <child link="rightfront_force_sensor"/>
@@ -505,9 +550,16 @@
     </joint>
     <link name="rightfront_force_sensor">
+      <!-- <pose>0.11 0.05 0.07 0 0 0</pose> -->
         <visual name="visual">
           <geometry>
             <box size="0.05 0.01 0.01"/>
           </geometry>
-        </visual>
+          <!-- <material>
+            <ambient>0 0 0 1</ambient>
+            <diffuse>0 0 0 1</diffuse>
+            <specular>0 0 0 0</specular>
+            <emissive>0 1 1 1</emissive>
+          </material>  -->
+        </visual><!---->
         <collision name="collision_rightfront_collision">
           <geometry>
@@ -515,6 +567,6 @@
           </geometry>
         </collision>
-    </link> -->
-    <!-- <joint name="leftfront_force_sensor_joint" type="fixed">
+    </link>
+    <joint name="leftfront_force_sensor_joint" type="fixed">
       <parent link="cube_base"/>
       <child link="leftfront_force_sensor"/>
@@ -522,9 +574,16 @@
     </joint>
     <link name="leftfront_force_sensor">
+      <!-- <pose>0.11 0.05 0.07 0 0 0</pose> -->
         <visual name="visual">
           <geometry>
             <box size="0.05 0.01 0.01"/>
           </geometry>
-        </visual>
+          <!-- <material>
+            <ambient>0 0 0 1</ambient>
+            <diffuse>0 0 0 1</diffuse>
+            <specular>0 0 0 0</specular>
+            <emissive>0 1 1 1</emissive>
+          </material>  -->
+        </visual><!---->
         <collision name="collision_leftfront_collision">
           <geometry>
@@ -532,6 +591,6 @@
           </geometry>
         </collision>
-    </link> -->
-    <!-- <joint name="LightSensor_joint" type="fixed">
+    </link>
+    <joint name="LightSensor_joint" type="fixed">
       <parent link="BaseBoards"/>
       <child link="LightSensor"/>
@@ -539,4 +598,5 @@
     </joint>
     <link name="LightSensor">
+      <!-- <pose>0.11 0.05 0.07 0 0 0</pose> -->
         <inertial>
           <origin xyz="0 0 0" />
@@ -551,5 +611,5 @@
             <mesh filename="package://myrobot/models/myroboturdf/meshes/Sensors/photodiode-Hamamatsu-S1223-01_BL.dae" scale="0.001 0.001 0.001"/>
           </geometry>
-        </visual>
+        </visual><!---->
         <collision name="collision">
           <geometry>
@@ -557,4 +617,7 @@
           </geometry>
         </collision>
+      <!-- <self_collide>0</self_collide>
+      <kinematic>0</kinematic>
+      <gravity>1</gravity> -->
     </link>
     <joint name="laser_sensor_joint" type="fixed">
@@ -564,4 +627,5 @@
     </joint>
     <link name="laser_sensor">
+      <!-- <pose>0.11 0.05 0.07 0 0 0</pose> -->
         <inertial>
           <origin xyz="0 0 0" />
@@ -577,4 +641,5 @@
         </collision>
     </link>
+    <!--%%%%%%%%%%%%%%%%%%%%%%%%%%%%%%%%%%%%%%%%%BOARDS%%%%%%%%%%%%%%%%%%%%%%%%%%%%%%%%%%%%%%%%%%%%%%-->
     <joint name="LattePanda_joint" type="fixed">
       <parent link="BaseBoards"/>
@@ -583,4 +648,5 @@
     </joint>
     <link name="LattePanda">
+      <!-- <pose>-0.012 0.001 0.153 0 0 0</pose> -->
       <inertial>
           <origin xyz="0 0 0" />
@@ -608,4 +674,5 @@
     </joint>
     <link name="K64F">
+      <!-- <pose>-0.012 0.001 0.153 0 0 0</pose> -->
       <inertial>
           <origin xyz="0 0 0" />
@@ -627,4 +694,5 @@
       </visual>
       </link>
+    <!--%%%%%%%%%%%%%%%%%%%%%%%%%%%%%%%%%%%%%%%%%MISCELLANEOUS%%%%%%%%%%%%%%%%%%%%%%%%%%%%%%%%%%%%%%%%%%%%%%-->
     <joint name="sg90h_joint" type="fixed">
       <parent link="supporto_sg90"/>
@@ -633,4 +701,5 @@
     </joint>
     <link name="sg90h">
+      <!-- <pose>-0.012 0.001 0.153 0 0 0</pose> -->
       <inertial>
           <origin xyz="0 0 0" />
@@ -659,4 +728,5 @@
     </joint>
     <link name="sg90h_shaft">
+      <!-- <pose>-0.012 0.001 0.153 0 0 0</pose> -->
       <inertial>
           <origin xyz="0 0 0" />
@@ -752,4 +822,170 @@
       </visual>
       </link>
-       -->
+    <!-- JOINTS -->
+    <!-- <joint type='revolute' name='left_wheel_hinge'>
+      <pose>0 0 -0.03 0 0 0</pose>
+      <child>left_wheel</child>
+      <parent>cube_base</parent>
+      <axis>
+        <xyz>0 0 1</xyz>
+      </axis>
+    </joint>
+    <joint type='revolute' name='right_wheel_hinge'>
+      <pose>0 0 0.03 0 0 0</pose>
+      <child>right_wheel</child>
+      <parent>cube_base</parent>
+      <axis>
+        <xyz>0 0 1</xyz>
+      </axis>
+    </joint>
+    <joint type='fixed' name='BaseBoards_joint'>
+      <pose>0 0 0 0 0 0</pose>
+      <child>BaseBoards</child>
+      <parent>cube_base</parent>
+    </joint>
+    <joint type='fixed' name='piastra_anteriore_joint'>
+      <pose>0 0 0 0 0 0</pose>
+      <child>piastra_anteriore</child>
+      <parent>cube_base</parent>
+    </joint>
+    <joint type='fixed' name='supporto_sg90_joint'>
+      <pose>0 0 0 0 0 0</pose>
+      <child>supporto_sg90</child>
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