Commit message: still not working well

File: models/myroboturdf/myrobot.urdf.xacro (robot description, xacro)
@@ -31,10 +31,10 @@
         </geometry>
       </visual>
-      <visual>
+      <!-- <visual>
         <origin xyz="0.02 0 -0.01" rpy="1.5707 0 1.5707"/>
         <geometry>
           <mesh filename="package://myrobot/models/myroboturdf/meshes/Devastator.dae"/>
         </geometry>
-      </visual>
+      </visual> -->
       <collision name = "caster_collision">
       <origin xyz="-0.05 0 -0.03" rpy="0 0 0"/>
@@ -149,16 +149,16 @@
         </geometry>
       </collision>
-      <visual>
+      <!-- <visual>
         <origin xyz="0.05 0 0" rpy="0 0 1.5707"/>
         <geometry>
           <mesh filename="package://myrobot/models/myroboturdf/meshes/Supports/BaseBoards.dae"/>
         </geometry>
-      </visual>
-       <!-- <visual>
+      </visual> -->
+       <visual>
         <origin xyz="0 0 0" rpy="0 0 0"/>
         <geometry>
           <box size="0.16 0.122315 0.002"/>
         </geometry>
-      </visual> -->
+      </visual>
       <collision name = "stick1_collision">
       <origin xyz="0.075 0.05 -0.02 " rpy="0 0 0"/>
@@ -227,16 +227,16 @@
         </geometry>
       </collision>
+      <visual>
+        <origin xyz="0 0 0 " rpy="0 0 0"/>
+        <geometry>
+          <box size="0.086 0.079320 0.003"/>
+        </geometry>
+      </visual>
       <!-- <visual>
-        <origin xyz="0 0 0 " rpy="0 0 0"/>
-        <geometry>
-          <box size="0.086 0.079320 0.003"/>
-        </geometry>
-      </visual>-->
-      <visual>
         <origin xyz="0.025 0 -0.0015 " rpy="0 0 1.5707"/>
         <geometry>
           <mesh filename="package://myrobot/models/myroboturdf/meshes/Supports/Piastra_anteriore2.dae"/>
         </geometry>
-      </visual>
+      </visual> -->
     </link>
     <joint name="supporto_sg90_joint" type="fixed">
@@ -257,16 +257,16 @@
         </geometry>
       </collision>
+      <!-- <visual>
+        <origin xyz="-0.003 0.015 0" rpy="0 0 1.5707"/>
+        <geometry>
+          <mesh filename="package://myrobot/models/myroboturdf/meshes/Supports/Supporto_sg90_base.dae"/>
+        </geometry>
+      </visual> -->
       <visual>
-        <origin xyz="-0.003 0.015 0" rpy="0 0 1.5707"/>
-        <geometry>
-          <mesh filename="package://myrobot/models/myroboturdf/meshes/Supports/Supporto_sg90_base.dae"/>
-        </geometry>
-      </visual>
-      <!-- <visual>
         <origin xyz="0 0 0 " rpy="0 0 0"/>
         <geometry>
           <box size="0.027 0.049 0.004"/>
         </geometry>
-      </visual> -->
+      </visual>
     </link>
     <joint name="supporto_piastra_albero_joint" type="fixed">
@@ -287,16 +287,16 @@
         </geometry>
       </collision>
+      <visual>
+        <origin xyz="0 0 0 " rpy="0 0 0"/>
+        <geometry>
+          <cylinder length="0.004" radius="0.008"/>
+        </geometry>
+      </visual>
       <!-- <visual>
-        <origin xyz="0 0 0 " rpy="0 0 0"/>
-        <geometry>
-          <cylinder length="0.004" radius="0.008"/>
+        <origin xyz="0 0 -0.002" rpy="1.5707 0 4.71238"/>
+        <geometry>
+          <mesh filename="package://myrobot/models/myroboturdf/meshes/Supports/Supporto_piastra_albero.dae" scale="1 1 1"/>
         </geometry>
       </visual> -->
-      <visual>
-        <origin xyz="0 0 -0.002" rpy="1.5707 0 4.71238"/>
-        <geometry>
-          <mesh filename="package://myrobot/models/myroboturdf/meshes/Supports/Supporto_piastra_albero.dae" scale="1 1 1"/>
-        </geometry>
-      </visual>
     </link>
     <!-- <joint name="supporto_pitch_servo_1_joint" type="fixed">
@@ -568,8 +568,14 @@
                    izz="2.0712558e-05" />
         </inertial>
+        <!-- <visual name="visual">
+          <origin xyz="0.001 0 0" rpy=" 0 0 -1.5707"/>
+          <geometry>
+            <mesh filename="package://myrobot/models/myroboturdf/meshes/Sensors/photodiode-Hamamatsu-S1223-01_BL.dae"/>
+          </geometry>
+        </visual> -->
         <visual name="visual">
           <origin xyz="0.001 0 0" rpy=" 0 0 -1.5707"/>
           <geometry>
-            <mesh filename="package://myrobot/models/myroboturdf/meshes/Sensors/photodiode-Hamamatsu-S1223-01_BL.dae"/>
+            <box size="0.005 0.01 0.01"/>
           </geometry>
         </visual>
@@ -602,5 +608,5 @@
       <parent link="BaseBoards"/>
       <child link="LattePanda"/>
-      <origin xyz="-0.012 0.001 0.0.002" rpy="0 0 0"/>
+      <origin xyz="-0.012 0.001 0.002" rpy="0 0 0"/>
     </joint>
     <link name="LattePanda">
@@ -617,15 +623,15 @@
           </geometry>
       </collision>
+      <visual name="visual">
+          <geometry>
+            <box size="0.12 0.08 0.01"/>
+          </geometry>
+      </visual>
       <!-- <visual name="visual">
-          <geometry>
-            <box size="0.12 0.08 0.01"/>
-          </geometry>
-      </visual>  -->
-      <visual name="visual">
           <origin xyz="0.001 0 0" rpy="1.5707 0 0 "/>
           <geometry>
             <mesh filename="package://myrobot/models/myroboturdf/meshes/Boards/LattePanda_delta.dae"/>
           </geometry>
-      </visual>
+      </visual> -->
       </link>
     <joint name="K64F_joint" type="fixed">
@@ -647,15 +653,15 @@
           </geometry>
       </collision>
+      <visual name="visual">
+          <geometry>
+            <box size="0.085 0.055 0.015"/>
+          </geometry>
+      </visual>
       <!-- <visual name="visual">
-          <geometry>
-            <box size="0.085 0.055 0.015"/>
-          </geometry>
-      </visual>   -->
-      <visual name="visual">
           <origin xyz="-0.037 -0.027 -0.007" rpy=" 0 0 0"/>
           <geometry>
             <mesh filename="package://myrobot/models/myroboturdf/meshes/Boards/K64F.dae"/>
           </geometry>
-      </visual>
+      </visual> -->
       </link>
     <joint name="sg90h_joint" type="fixed">
@@ -682,10 +688,10 @@
           </geometry>
       </visual>
-      <visual name="visual">
+      <!-- <visual name="visual">
           <origin xyz="0 -0.011 0" rpy=" 0 0 0"/>
           <geometry>
             <mesh filename="package://myrobot/models/myroboturdf/meshes/Misc/sg90.dae"/>
           </geometry>
-      </visual>
+      </visual> -->
       </link>
     <joint name="sg90h_shaft_joint" type="continuous">

Commit message: working slam!

File: models/myroboturdf/myrobot.urdf.xacro (robot description, xacro)
@@ -267,5 +267,5 @@
       </visual>
     </link>
-    <joint name="supporto_piastra_albero_joint" type="fixed">
+   <!--  <joint name="supporto_piastra_albero_joint" type="fixed">
       <parent link="sg90h_shaft"/>
       <child link="supporto_piastra_albero"/>
@@ -290,11 +290,11 @@
         </geometry>
       </visual>
-      <!-- <visual name="supporto_piastra_albero_visual">
+      <visual name="supporto_piastra_albero_visual">
         <origin xyz="0 0 -0.002" rpy="1.5707 0 4.71238"/>
         <geometry>
           <mesh filename="package://myrobot/models/myroboturdf/meshes/Supports/Supporto_piastra_albero.dae" scale="1 1 1"/>
         </geometry>
-      </visual> -->
-    </link>
+      </visual>
+    </link>-->
     <!-- <joint name="supporto_pitch_servo_1_joint" type="fixed">
       <parent link="supporto_piastra_albero"/>
@@ -692,5 +692,5 @@
       </visual> -->
       </link>
-    <joint name="sg90h_shaft_joint" type="continuous">
+    <!-- <joint name="sg90h_shaft_joint" type="continuous">
       <parent link="sg90h"/>
       <child link="sg90h_shaft"/>
@@ -716,5 +716,5 @@
         </geometry>
       </visual>
-    </link>
+    </link> -->
     <!-- <joint name="sg90v_joint" type="fixed">
       <parent link="supporto_pitch_servo_2"/>

Commit message: added stl files (other need conversion)

File: models/myroboturdf/myrobot.urdf.xacro (robot description, xacro)
@@ -23,15 +23,15 @@
         </geometry>
       </collision>
-     <visual name="cube_base_visual">
+     <!-- <visual name="cube_base_visual">
         <geometry>
           <box size="0.19 0.134 0.047"/>
         </geometry>
-      </visual>
-      <!-- <visual>
+      </visual> -->
+      <visual name="cube_base_visual">
         <origin xyz="0.02 0 -0.01" rpy="1.5707 0 1.5707"/>
         <geometry>
-          <mesh filename="package://myrobot/models/myroboturdf/meshes/Devastator.dae"/>
-        </geometry>
-      </visual> -->
+          <mesh filename="package://myrobot/models/myroboturdf/meshes/Devastator.stl" scale="0.001 0.001 0.001"/>
+        </geometry>
+      </visual>
       <collision name = "caster_collision">
       <origin xyz="-0.05 0 -0.03" rpy="0 0 0"/>
@@ -50,10 +50,10 @@
         </surface>
       </collision>
-      <visual name="caster_visual">
+      <!-- <visual name="caster_visual">
       <origin xyz="-0.05 0 -0.03" rpy="0 0 0"/>
         <geometry>
           <sphere radius="0.05"/>
         </geometry>
-      </visual>
+      </visual> -->
       <collision name = 'caster2_collision'>
       <origin xyz="0.05 0 -0.03" rpy="0 0 0"/>
@@ -72,10 +72,10 @@
         </surface>
       </collision>
-      <visual name="caster2_visual">
+     <!-- <visual name="caster2_visual">
       <origin xyz="0.05 0 -0.03" rpy="0 0 0"/>
         <geometry>
           <sphere radius="0.05"/>
         </geometry>
-      </visual>
+      </visual> -->
     </link>
     <joint name="wheel_left_joint" type="continuous">
@@ -92,15 +92,14 @@
       </inertial>
       <collision name="wheel_left_link_collision">
-        <!-- <origin xyz="0 0 0" rpy="0 0 0"/> -->
         <geometry>
           <cylinder length="0.035" radius="0.06"/>
         </geometry>
       </collision>
-      <visual name="wheel_left_link_visual">
+      <!-- <visual name="wheel_left_link_visual">
         <origin xyz="0 0 0" rpy="0 0 0"/>
         <geometry>
           <cylinder length="0.035" radius="0.06"/>
         </geometry>
-      </visual>
+      </visual> -->
     </link>
     <joint name="wheel_right_joint" type="continuous">
@@ -117,15 +116,14 @@
       </inertial>
       <collision name="wheel_right_link_collision">
-        <!-- <origin xyz="0 0 0" rpy="0 0 0"/> -->
         <geometry>
           <cylinder length="0.035" radius="0.06"/>
         </geometry>
       </collision>
-      <visual name="wheel_right_link_visual">
+      <!-- <visual name="wheel_right_link_visual">
         <origin xyz="0 0 0" rpy="0 0 0"/>
         <geometry>
           <cylinder length="0.035" radius="0.06"/>
         </geometry>
-      </visual>
+      </visual> -->
     </link>
     <joint name="BaseBoards_joint" type="fixed">
@@ -141,16 +139,16 @@
         </geometry>
       </collision>
-      <!-- <visual  name="BaseBoards_visual">
+      <visual  name="BaseBoards_visual">
         <origin xyz="0.05 0 0" rpy="0 0 1.5707"/>
         <geometry>
-          <mesh filename="package://myrobot/models/myroboturdf/meshes/Supports/BaseBoards.dae"/>
-        </geometry>
-      </visual> -->
-       <visual name="BaseBoards_visual">
+          <mesh filename="package://myrobot/models/myroboturdf/meshes/Supports/BaseBoards.STL" scale="0.001 0.001 0.001"/>
+        </geometry>
+      </visual>
+       <!-- <visual name="BaseBoards_visual">
         <origin xyz="0 0 0" rpy="0 0 0"/>
         <geometry>
           <box size="0.16 0.122315 0.002"/>
         </geometry>
-      </visual>
+      </visual> -->
       <collision name = "stick1_collision">
       <origin xyz="0.075 0.05 -0.02 " rpy="0 0 0"/>
@@ -220,10 +218,10 @@
         </geometry>
       </visual>
-      <!-- <visual>
+      <visual>
         <origin xyz="0.025 0 -0.0015 " rpy="0 0 1.5707"/>
         <geometry>
-          <mesh filename="package://myrobot/models/myroboturdf/meshes/Supports/Piastra_anteriore2.dae"/>
-        </geometry>
-      </visual> -->
+          <mesh filename="package://myrobot/models/myroboturdf/meshes/Supports/Piastra_anteriore2.stl"/>
+        </geometry>
+      </visual>
     </link>
     <joint name="supporto_sg90_joint" type="fixed">

Commit message: comments added, model in collision mode

File: models/myroboturdf/myrobot.urdf.xacro (robot description, xacro)
@@ -29,9 +29,10 @@
         </geometry>
       </collision>
-     <!-- <visual name="cube_base_visual">
+     <visual name="cube_base_visual">
         <geometry>
           <box size="0.19 0.134 0.047"/>
         </geometry>
-      </visual> -->
+      </visual>
+<!--
       <visual name="cube_base_visual">
         <origin xyz="0.02 0 -0.01" rpy="1.5707 0 1.5707"/>
@@ -40,5 +41,5 @@
         </geometry>
         <material name="light_black"/>
-      </visual>
+      </visual> -->
       <collision name = "caster_collision">
       <origin xyz="-0.05 0 -0.03" rpy="0 0 0"/>
@@ -57,10 +58,10 @@
         </surface>
       </collision>
-      <!-- <visual name="caster_visual">
+      <visual name="caster_visual">
       <origin xyz="-0.05 0 -0.03" rpy="0 0 0"/>
         <geometry>
           <sphere radius="0.05"/>
         </geometry>
-      </visual> -->
+      </visual>
       <collision name = 'caster2_collision'>
       <origin xyz="0.05 0 -0.03" rpy="0 0 0"/>
@@ -79,10 +80,10 @@
         </surface>
       </collision>
-     <!-- <visual name="caster2_visual">
+     <visual name="caster2_visual">
       <origin xyz="0.05 0 -0.03" rpy="0 0 0"/>
         <geometry>
           <sphere radius="0.05"/>
         </geometry>
-      </visual> -->
+      </visual>
     </link>
 <!--
@@ -129,10 +130,10 @@
         </geometry>
       </collision>
-      <!-- <visual name="wheel_left_link_visual">
+      <visual name="wheel_left_link_visual">
         <origin xyz="0 0 0" rpy="0 0 0"/>
         <geometry>
           <cylinder length="0.035" radius="0.06825"/>
         </geometry>
-      </visual> -->
+      </visual>
     </link>
     <joint name="wheel_right_joint" type="continuous">
@@ -153,10 +154,10 @@
         </geometry>
       </collision>
-      <!-- <visual name="wheel_right_link_visual">
+      <visual name="wheel_right_link_visual">
         <origin xyz="0 0 0" rpy="0 0 0"/>
         <geometry>
           <cylinder length="0.035" radius="0.06825"/>
         </geometry>
-      </visual> -->
+      </visual>
     </link>
     <joint name="BaseBoards_joint" type="fixed">
