Commit message: model is all visual now

File: models/myroboturdf/myrobot.urdf.xacro (robot description, xacro)
@@ -29,10 +29,9 @@
         </geometry>
       </collision>
-     <visual name="cube_base_visual">
+     <!-- <visual name="cube_base_visual">
         <geometry>
           <box size="0.19 0.134 0.047"/>
         </geometry>
-      </visual>
-<!--
+      </visual> -->
       <visual name="cube_base_visual">
         <origin xyz="0.02 0 -0.01" rpy="1.5707 0 1.5707"/>
@@ -41,5 +40,5 @@
         </geometry>
         <material name="light_black"/>
-      </visual> -->
+      </visual>
       <collision name = "caster_collision">
       <origin xyz="-0.05 0 -0.03" rpy="0 0 0"/>
@@ -58,4 +57,5 @@
         </surface>
       </collision>
+<!--
       <visual name="caster_visual">
       <origin xyz="-0.05 0 -0.03" rpy="0 0 0"/>
@@ -63,5 +63,5 @@
           <sphere radius="0.05"/>
         </geometry>
-      </visual>
+      </visual> -->
       <collision name = 'caster2_collision'>
       <origin xyz="0.05 0 -0.03" rpy="0 0 0"/>
@@ -80,10 +80,10 @@
         </surface>
       </collision>
-     <visual name="caster2_visual">
+     <!-- <visual name="caster2_visual">
       <origin xyz="0.05 0 -0.03" rpy="0 0 0"/>
         <geometry>
           <sphere radius="0.05"/>
         </geometry>
-      </visual>
+      </visual> -->
     </link>
 <!--
@@ -130,10 +130,10 @@
         </geometry>
       </collision>
-      <visual name="wheel_left_link_visual">
+      <!-- <visual name="wheel_left_link_visual">
         <origin xyz="0 0 0" rpy="0 0 0"/>
         <geometry>
           <cylinder length="0.035" radius="0.06825"/>
         </geometry>
-      </visual>
+      </visual> -->
     </link>
     <joint name="wheel_right_joint" type="continuous">
@@ -154,10 +154,10 @@
         </geometry>
       </collision>
-      <visual name="wheel_right_link_visual">
+      <!--<visual  name="wheel_right_link_visual">
         <origin xyz="0 0 0" rpy="0 0 0"/>
         <geometry>
           <cylinder length="0.035" radius="0.06825"/>
         </geometry>
-      </visual>
+      </visual>-->
     </link>
     <joint name="BaseBoards_joint" type="fixed">
@@ -173,5 +173,5 @@
         </geometry>
       </collision>
-      <!-- <visual  name="BaseBoards_visual">
+      <visual  name="BaseBoards_visual">
         <origin xyz="0.05 0 0" rpy="0 0 1.5707"/>
         <geometry>
@@ -179,11 +179,11 @@
         </geometry>
         <material name="blue"/>
-      </visual> -->
-       <visual name="BaseBoards_visual">
+      </visual>
+       <!-- <visual name="BaseBoards_visual">
         <origin xyz="0 0 0" rpy="0 0 0"/>
         <geometry>
           <box size="0.16 0.122315 0.002"/>
         </geometry>
-      </visual>
+      </visual> -->
       <collision name = "stick1_collision">
       <origin xyz="0.075 0.05 -0.02 " rpy="0 0 0"/>
@@ -251,11 +251,11 @@
         </geometry>
       </collision>
-      <visual name ="piastra_anteriore_visual">
+      <!-- <visual name ="piastra_anteriore_visual">
         <origin xyz="0 0 0 " rpy="0 0 0"/>
         <geometry>
           <box size="0.086 0.079320 0.003"/>
         </geometry>
-      </visual>
-      <!-- <visual>
+      </visual> -->
+      <visual>
         <origin xyz="0.025 0 -0.0015 " rpy="0 0 1.5707"/>
         <geometry>
@@ -263,5 +263,5 @@
         </geometry>
         <material name="grey"/>
-      </visual> -->
+      </visual>
     </link>
     <joint name="supporto_sg90_joint" type="fixed">
@@ -277,16 +277,16 @@
         </geometry>
       </collision>
-      <!-- <visual>
+      <visual>
         <origin xyz="-0.003 0.015 0" rpy="0 0 1.5707"/>
         <geometry>
           <mesh filename="package://myrobot/models/myroboturdf/meshes/Supports/Supporto_sg90_base.stl" scale="0.001 0.001 0.001"/>
         </geometry>
-      </visual> -->
-      <visual name="supporto_sg90_visual">
+      </visual>
+      <!-- <visual name="supporto_sg90_visual">
         <origin xyz="0 0 0 " rpy="0 0 0"/>
         <geometry>
           <box size="0.027 0.049 0.004"/>
         </geometry>
-      </visual>
+      </visual> -->
     </link>
     <joint name="supporto_piastra_albero_joint" type="fixed">
@@ -302,16 +302,16 @@
         </geometry>
       </collision>
+      <!-- <visual name="supporto_piastra_albero_visual">
+        <origin xyz="0 0 0 " rpy="0 0 0"/>
+        <geometry>
+          <cylinder length="0.004" radius="0.008"/>
+        </geometry>
+      </visual> -->
       <visual name="supporto_piastra_albero_visual">
-        <origin xyz="0 0 0 " rpy="0 0 0"/>
-        <geometry>
-          <cylinder length="0.004" radius="0.008"/>
-        </geometry>
-      </visual>
-      <!-- <visual name="supporto_piastra_albero_visual">
         <origin xyz="0 0 -0.002" rpy="1.5707 0 4.71238"/>
         <geometry>
           <mesh filename="package://myrobot/models/myroboturdf/meshes/Supports/Supporto_piastra_albero.stl" scale="0.001 0.001 0.001"/>
         </geometry>
-      </visual>  -->
+      </visual>
     </link>
     <joint name="supporto_pitch_servo_1_joint" type="fixed">
@@ -326,15 +326,15 @@
         </geometry>
       </collision>
-      <visual name="supporto_pitch_servo_1_visual">
+      <!-- <visual name="supporto_pitch_servo_1_visual">
         <geometry>
           <box size="0.035 0.12 0.003"/>
         </geometry>
-      </visual>
-      <!-- <visual name='supporto_pitch_servo_1_visual'>
+      </visual>  -->
+      <visual name='supporto_pitch_servo_1_visual'>
       <origin xyz="0 0 0.004" rpy="3.1415 0 1.5707" />
         <geometry>
           <mesh filename="package://myrobot/models/myroboturdf/meshes/Supports/supporto_pitch_servo_1_new.stl" scale="0.001 0.001 0.001"/>
         </geometry>
-      </visual> -->
+      </visual>
     </link>
     <joint name="supporto_pitch_servo_2_joint" type="fixed">
@@ -349,15 +349,15 @@
         </geometry>
       </collision>
+      <visual name='supporto_pitch_servo_2_visual'>
+      <origin xyz="-0.042 0 0.02" rpy="0 3.1415 0" />
+        <geometry>
+          <mesh filename="package://myrobot/models/myroboturdf/meshes/Supports/supporto_pitch_servo_2.stl" scale="0.001 0.001 0.001"/>
+        </geometry>
+      </visual>
       <!-- <visual name='supporto_pitch_servo_2_visual'>
-      <origin xyz="-0.042 0 0.02" rpy="0 3.1415 0" />
-        <geometry>
-          <mesh filename="package://myrobot/models/myroboturdf/meshes/Supports/supporto_pitch_servo_2.stl" scale="0.001 0.001 0.001"/>
-        </geometry>
-      </visual> -->
-      <visual name='supporto_pitch_servo_2_visual'>
         <geometry>
           <box size="0.002 0.02 0.035"/>
         </geometry>
-      </visual>
+      </visual>  -->
     </link>
     <joint name="supporto_pitch_servo_2_noservo_joint" type="fixed">
@@ -372,5 +372,5 @@
         </geometry>
       </collision>
-      <!-- <visual name='supporto_pitch_servo_2_noservo_visual'>
+      <visual name='supporto_pitch_servo_2_noservo_visual'>
       <origin xyz="0.085 0 0.02" rpy="0 3.1415 0" />
         <geometry>
@@ -378,10 +378,10 @@
             scale="0.001 0.001 0.001"/>
         </geometry>
-      </visual> -->
-      <visual name='supporto_pitch_servo_2_noservo_visual'>
+      </visual>
+      <!-- <visual name='supporto_pitch_servo_2_noservo_visual'>
         <geometry>
           <box size="0.002 0.019 0.036"/>
         </geometry>
-      </visual>
+      </visual> -->
     </link>
     <joint name="supp_RS_joint" type="fixed">
@@ -396,15 +396,15 @@
         </geometry>
       </collision>
-      <!-- <visual name='supp_RS_visual'>
+      <visual name='supp_RS_visual'>
      <origin xyz="0.0 0.054 0.013" rpy="1.5707 0 1.5707"/>
         <geometry>
           <mesh filename="package://myrobot/models/myroboturdf/meshes/Supports/Supp_RS.dae"/>
         </geometry>
-      </visual>  -->
-      <visual name='visuall'>
+      </visual>
+      <!-- <visual name='visuall'>
         <geometry>
           <box size="0.016 0.105 0.0035"/>
         </geometry>
-      </visual>
+      </visual> -->
       <collision name='vertical3_collision'>
       <origin xyz="0 0.05 0.01" rpy="0 0 0"/>
@@ -413,10 +413,10 @@
         </geometry>
       </collision>
-      <visual name='vertical3_visual'>
+      <!-- <visual name='vertical3_visual'>
       <origin xyz="0 0.05 0.01" rpy="0 0 0"/>
         <geometry>
           <box size="0.016 0.0035 0.02"/>
         </geometry>
-      </visual>
+      </visual> -->
       <collision name='vertical4_collision'>
       <origin xyz="0 -0.05 0.01" rpy="0 0 0"/>
@@ -425,10 +425,10 @@
         </geometry>
       </collision>
-      <visual name='vertical4_visual'>
+      <!-- <visual name='vertical4_visual'>
       <origin xyz="0 -0.05 0.01" rpy="0 0 0"/>
         <geometry>
           <box size="0.016 0.0035 0.02"/>
         </geometry>
-      </visual>
+      </visual>-->
     </link>
   <joint name="imu_joint" type="fixed">
@@ -449,17 +449,17 @@
           </geometry>
         </collision>
-        <visual name="RealSense_visual2">
+        <!-- <visual name="RealSense_visual2">
           <geometry>
             <box size="0.025 0.087 0.02"/>
+          </geometry>
+          <material name="white"/>
+        </visual> -->
+        <visual name="RealSense_visual">
+          <origin xyz="0.0125 0.0 0" rpy="1.5707 0 1.5707"/>
+          <geometry>
+            <mesh filename="package://myrobot/models/myroboturdf/meshes/Sensors/IntelRealsense_D435_Multibody.dae"/>
           </geometry>
           <material name="white"/>
         </visual>
-        <!-- <visual name="RealSense_visual">
-          <origin xyz="0.0125 0.0 0" rpy="1.5707 0 1.5707"/>
-          <geometry>
-            <mesh filename="package://myrobot/models/myroboturdf/meshes/Sensors/IntelRealsense_D435_Multibody.dae"/>
-          </geometry>
-          <material name="white"/>
-        </visual> -->
     </link>
     <joint name="rightfront_force_sensor_joint" type="fixed">
@@ -558,15 +558,15 @@
           </geometry>
       </collision>
+      <!-- <visual name="LattePanda_visual">
+          <geometry>
+            <box size="0.12 0.08 0.01"/>
+          </geometry>
+      </visual>  -->
       <visual name="LattePanda_visual">
-          <geometry>
-            <box size="0.12 0.08 0.01"/>
-          </geometry>
-      </visual>
-      <!-- <visual name="LattePanda_visual">
           <origin xyz="0.001 0 0" rpy="1.5707 0 0 "/>
           <geometry>
             <mesh filename="package://myrobot/models/myroboturdf/meshes/Boards/LattePanda_delta.dae"/>
           </geometry>
-      </visual> -->
+      </visual>
       </link>
     <joint name="K64F_joint" type="fixed">
@@ -581,15 +581,15 @@
           </geometry>
       </collision>
-      <visual name="K64F_visual">
+      <!-- <visual name="K64F_visual">
           <geometry>
             <box size="0.085 0.055 0.015"/>
           </geometry>
-      </visual>
-      <!-- <visual name="visual">
+      </visual>   -->
+      <visual name="visual">
           <origin xyz="-0.037 -0.027 -0.007" rpy=" 0 0 0"/>
           <geometry>
             <mesh filename="package://myrobot/models/myroboturdf/meshes/Boards/K64F.dae"/>
           </geometry>
-      </visual> -->
+      </visual>
       </link>
     <joint name="sg90h_joint" type="fixed">
@@ -611,15 +611,15 @@
           </geometry>
       </collision>
+      <!-- <visual name="sg90h_visual">
+          <geometry>
+            <box size=".012 0.022 0.022"/>
+          </geometry>
+      </visual>  -->
       <visual name="sg90h_visual">
-          <geometry>
-            <box size=".012 0.022 0.022"/>
-          </geometry>
-      </visual>
-      <!-- <visual name="sg90h_visual">
           <origin xyz="0 -0.011 0" rpy=" 0 0 0"/>
           <geometry>
             <mesh filename="package://myrobot/models/myroboturdf/meshes/Misc/sg90.dae"/>
           </geometry>
-      </visual> -->
+      </visual>
     </link>
     <joint name="sg90h_shaft_joint" type="fixed">
@@ -666,15 +666,15 @@
           </geometry>
       </collision>
-      <visual name="sg90v_visual">
+      <!-- <visual name="sg90v_visual">
           <geometry>
             <box size=".012 0.022 0.022"/>
           </geometry>
-      </visual>
-       <!-- <visual name="sg90v_visual">
+      </visual> -->
+       <visual name="sg90v_visual">
           <origin xyz="0 -0.011 0" rpy=" 0 0 0"/>
           <geometry>
             <mesh filename="package://myrobot/models/myroboturdf/meshes/Misc/sg90.dae"/>
           </geometry>
-      </visual>  -->
+      </visual>
       </link>
     <joint name="sg90v_shaft_joint" type="fixed">
@@ -714,15 +714,15 @@
           </geometry>
       </collision>
+      <!-- <visual name="batteria_visual">
+          <geometry>
+            <box size="0.102 0.035 0.025"/>
+          </geometry>
+      </visual>  -->
       <visual name="batteria_visual">
-          <geometry>
-            <box size="0.102 0.035 0.025"/>
-          </geometry>
-      </visual>
-      <!-- <visual name="batteria_visual">
           <origin xyz="0 0 -0.012" rpy=" 0 0 0"/>
           <geometry>
             <mesh filename="package://myrobot/models/myroboturdf/meshes/Misc/Turnigy_2200mAh_3S_20C_Lipo_Pack.dae"/>
           </geometry>
-      </visual> -->
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
Commit message: added a node that transforms odometry (set_odom.py)

File: models/myroboturdf/myrobot.urdf.xacro (robot description, xacro)
@@ -29,10 +29,10 @@
         </geometry>
       </collision>
-     <visual name="cube_base_visual">
+     <!-- <visual name="cube_base_visual">
         <geometry>
           <box size="0.19 0.134 0.047"/>
         </geometry>
-      </visual>
-      <!-- <visual name="cube_base_visual">
+      </visual> -->
+      <visual name="cube_base_visual">
         <origin xyz="0.02 0 -0.01" rpy="1.5707 0 1.5707"/>
         <geometry>
@@ -40,5 +40,5 @@
         </geometry>
         <material name="light_black"/>
-      </visual> -->
+      </visual>
       <collision name = "caster_collision">
       <origin xyz="-0.05 0 -0.03" rpy="0 0 0"/>
@@ -57,5 +57,5 @@
         </surface>
       </collision>
-      <visual name="caster_visual">
+      <!-- <visual name="caster_visual">
       <origin xyz="-0.05 0 -0.03" rpy="0 0 0"/>
         <geometry>
@@ -63,4 +63,5 @@
         </geometry>
       </visual>
+       -->
       <collision name = 'caster2_collision'>
       <origin xyz="0.05 0 -0.03" rpy="0 0 0"/>
@@ -79,10 +80,10 @@
         </surface>
       </collision>
-     <visual name="caster2_visual">
+     <!-- <visual name="caster2_visual">
       <origin xyz="0.05 0 -0.03" rpy="0 0 0"/>
         <geometry>
           <sphere radius="0.05"/>
         </geometry>
-      </visual>
+      </visual> -->
     </link>
 <!--
@@ -129,10 +130,10 @@
         </geometry>
       </collision>
-      <visual name="wheel_left_link_visual">
+      <!-- <visual name="wheel_left_link_visual">
         <origin xyz="0 0 0" rpy="0 0 0"/>
         <geometry>
           <cylinder length="0.035" radius="0.06825"/>
         </geometry>
-      </visual>
+      </visual> -->
     </link>
     <joint name="wheel_right_joint" type="continuous">
@@ -153,10 +154,10 @@
         </geometry>
       </collision>
-      <visual  name="wheel_right_link_visual">
+      <!-- <visual  name="wheel_right_link_visual">
         <origin xyz="0 0 0" rpy="0 0 0"/>
         <geometry>
           <cylinder length="0.035" radius="0.06825"/>
         </geometry>
-      </visual>
+      </visual> -->
     </link>
     <joint name="BaseBoards_joint" type="fixed">
