Commit message: mounting the model slowly

File: models/myroboturdf/myrobot.gazebo.xacro (robot description, xacro)
@@ -37,5 +37,5 @@
       </camera>
     </sensor>
-  </gazebo>
+  </gazebo>-->
   <gazebo reference="rightfront_force_sensor">
     <sensor name="rf_force_sensor" type="contact">
@@ -56,5 +56,5 @@
     </sensor>
   </gazebo>
-  <gazebo reference="LightSensor">
+<gazebo reference="LightSensor">
     <sensor name='camera' type='depth'>
       <camera name='camera'>
@@ -96,5 +96,5 @@
       </ray>
     </sensor>
-  </gazebo> -->
+  </gazebo>
 <!-- PLUGINS -->
   <!-- <gazebo>
@@ -125,5 +125,5 @@
   </gazebo> -->
   <!-- <gazebo>
-    <plugin name="gazebo_ros_bumper_controller" filename="libcontact_plugin.so">
+    <plugin name="gazebo_right_bumper_controller" filename="libcontact_plugin.so">
       <alwaysOn>true</alwaysOn>
       <updateRate>30.0</updateRate>
@@ -133,5 +133,5 @@
   </gazebo>
   <gazebo>
-    <plugin name="gazebo_ros_bumper_controller" filename="libcontact_plugin.so">
+    <plugin name="gazebo_left_bumper_controller" filename="libcontact_plugin.so">
       <alwaysOn>true</alwaysOn>
       <updateRate>30.0</updateRate>
@@ -141,5 +141,5 @@
   </gazebo> -->
   <!-- <gazebo>
-    <plugin name="myrobot" filename="liblight_sensor_plugin.so">
+    <plugin name="light_sensor_plugin" filename="liblight_sensor_plugin.so">
       <cameraName>camera2</cameraName>
       <alwaysOn>true</alwaysOn>
@@ -159,5 +159,5 @@
       <distortion_t2>0.0</distortion_t2>
       <pointCloudCutoff>0.4</pointCloudCutoff>
-      <robotNamespace>/</robotNamespace>
+      <robotNamespace>base_footprint</robotNamespace>
     </plugin>
   </gazebo> -->
@@ -165,5 +165,5 @@
     <plugin name="gazebo_ros_lds_lfcd_controller" filename="libgazebo_ros_laser.so">
       <topicName>scan</topicName>
-      <frameName>cube_base</frameName>
+      <frameName>laser_scan</frameName>
     </plugin>
   </gazebo> -->

File: models/myroboturdf/myrobot.urdf.xacro (robot description, xacro)
@@ -31,10 +31,10 @@
         </geometry>
       </visual>
-      <!-- <visual>
+      <visual>
         <origin xyz="0.02 0 -0.01" rpy="1.5707 0 1.5707"/>
         <geometry>
           <mesh filename="package://myrobot/models/myroboturdf/meshes/Devastator.dae"/>
         </geometry>
-      </visual> -->
+      </visual>
       <collision name = "caster_collision">
       <origin xyz="-0.05 0 -0.03" rpy="0 0 0"/>
@@ -85,6 +85,6 @@
       <parent link="cube_base"/>
       <child link="wheel_left_link"/>
-      <origin xyz="0. 0.087 0.06825" rpy="0 1.5707 1.5707"/>
-      <axis xyz="0 0 1"/>
+      <origin xyz="0. 0.087 -0.011" rpy="0 1.5707 1.5707"/>
+      <axis xyz="1 0 0"/>
     </joint>
     <link name="wheel_left_link">
@@ -110,6 +110,6 @@
       <parent link="cube_base"/>
       <child link="wheel_right_link"/>
-      <origin xyz="0. -0.087 0.06825" rpy="0 0 0"/>
-      <axis xyz="0 0 1"/>
+      <origin xyz="0. -0.087 -0.011" rpy="0 0 0"/>
+      <axis xyz="1 0 0"/>
     </joint>
     <link name="wheel_right_link">
@@ -132,8 +132,8 @@
       </visual>
     </link>
-    <!-- <joint name="BaseBoards_joint" type="fixed">
+    <joint name="BaseBoards_joint" type="fixed">
       <parent link="cube_base"/>
       <child link="BaseBoards"/>
-      <origin xyz="-0.01 0 0.1435" rpy="0 0 0"/>
+      <origin xyz="-0.01 0 0.0635" rpy="0 0 0"/>
     </joint>
     <link name="BaseBoards">
@@ -155,4 +155,10 @@
         </geometry>
       </visual>
+       <visual>
+        <origin xyz="0 0 0" rpy="0 0 0"/>
+        <geometry>
+          <box size="0.16 0.122315 0.002"/>
+        </geometry>
+      </visual>
       <collision name = "stick1_collision">
       <origin xyz="0.075 0.05 -0.02 " rpy="0 0 0"/>
@@ -204,9 +210,8 @@
       </visual>
     </link>
-     -->
-    <!-- <joint name="piastra_anteriore_joint" type="fixed">
-      <parent link="BaseBoards"/>
+    <joint name="piastra_anteriore_joint" type="fixed">
+      <parent link="cube_base"/>
       <child link="piastra_anteriore"/>
-      <origin xyz="0.078 -0.004 0.104" rpy="0 0 0"/>
+      <origin xyz="0.078 -0.004 0.024" rpy="0 0 0"/>
     </joint>
     <link name="piastra_anteriore">
@@ -222,15 +227,21 @@
         </geometry>
       </collision>
+      <!-- <visual>
+        <origin xyz="0 0 0 " rpy="0 0 0"/>
+        <geometry>
+          <box size="0.086 0.079320 0.003"/>
+        </geometry>
+      </visual>-->
       <visual>
         <origin xyz="0.025 0 -0.0015 " rpy="0 0 1.5707"/>
         <geometry>
-          <mesh filename="package:/myrobot/models/myroboturdf/meshes/Supports/Piastra_anteriore2.dae" scale="1 1 1"/>
-        </geometry>
-      </visual>
-    </link> -->
-    <!-- <joint name="supporto_sg90_joint" type="fixed">
+          <mesh filename="package://myrobot/models/myroboturdf/meshes/Supports/Piastra_anteriore2.dae"/>
+        </geometry>
+      </visual>
+    </link>
+    <joint name="supporto_sg90_joint" type="fixed">
       <parent link="piastra_anteriore"/>
       <child link="supporto_sg90"/>
-      <origin xyz="0.094 -0.004 0.0995" rpy="0 0 0"/>
+      <origin xyz="0.024 0 -0.005" rpy="0 0 0"/>
     </joint>
     <link name="supporto_sg90">
@@ -249,9 +260,14 @@
         <origin xyz="-0.003 0.015 0" rpy="0 0 1.5707"/>
         <geometry>
-          <mesh filename="package://myrobot/models/myroboturdf/meshes/Supports/Supporto_sg90_base.dae" scale="1 1 1"/>
-        </geometry>
-      </visual>
-    </link>
-     -->
+          <mesh filename="package://myrobot/models/myroboturdf/meshes/Supports/Supporto_sg90_base.dae"/>
+        </geometry>
+      </visual>
+      <!-- <visual>
+        <origin xyz="0 0 0 " rpy="0 0 0"/>
+        <geometry>
+          <box size="0.027 0.049 0.004"/>
+        </geometry>
+      </visual> -->
+    </link>
     <!-- <joint name="supporto_piastra_albero_joint" type="fixed">
       <parent link="sg90h_shaft"/>
@@ -499,8 +515,8 @@
         </visual>
     </link> -->
-    <!-- <joint name="rightfront_force_sensor_joint" type="fixed">
+    <joint name="rightfront_force_sensor_joint" type="fixed">
       <parent link="cube_base"/>
       <child link="rightfront_force_sensor"/>
-      <origin xyz="0.11 0.05 0.07" rpy="0 0 0"/>
+      <origin xyz="0.11 0.05 0" rpy="0 0 0"/>
     </joint>
     <link name="rightfront_force_sensor">
@@ -515,9 +531,9 @@
           </geometry>
         </collision>
-    </link> -->
-    <!-- <joint name="leftfront_force_sensor_joint" type="fixed">
+    </link>
+    <joint name="leftfront_force_sensor_joint" type="fixed">
       <parent link="cube_base"/>
       <child link="leftfront_force_sensor"/>
-      <origin xyz="0.11 -0.05 0.07" rpy="0 0 0"/>
+      <origin xyz="0.11 -0.05 0" rpy="0 0 0"/>
     </joint>
     <link name="leftfront_force_sensor">
@@ -532,9 +548,9 @@
           </geometry>
         </collision>
-    </link> -->
-    <!-- <joint name="LightSensor_joint" type="fixed">
+    </link>
+    <joint name="LightSensor_joint" type="fixed">
       <parent link="BaseBoards"/>
       <child link="LightSensor"/>
-      <origin xyz="0.055 0.04 0.153 " rpy="0 -1.5707 0"/>
+      <origin xyz="0.055 0.04 0.008 " rpy="0 -1.5707 0"/>
     </joint>
     <link name="LightSensor">
@@ -549,5 +565,5 @@
           <origin xyz="0.001 0 0" rpy=" 0 0 -1.5707"/>
           <geometry>
-            <mesh filename="package://myrobot/models/myroboturdf/meshes/Sensors/photodiode-Hamamatsu-S1223-01_BL.dae" scale="0.001 0.001 0.001"/>
+            <mesh filename="package://myrobot/models/myroboturdf/meshes/Sensors/photodiode-Hamamatsu-S1223-01_BL.dae"/>
           </geometry>
         </visual>
@@ -580,5 +596,5 @@
       <parent link="BaseBoards"/>
       <child link="LattePanda"/>
-      <origin xyz="-0.012 0.001 0.153" rpy="0 0 0"/>
+      <origin xyz="-0.012 0.001 0.0.002" rpy="0 0 0"/>
     </joint>
     <link name="LattePanda">
@@ -595,8 +611,13 @@
           </geometry>
       </collision>
+      <!-- <visual name="visual">
+          <geometry>
+            <box size="0.12 0.08 0.01"/>
+          </geometry>
+      </visual>  -->
       <visual name="visual">
-          <origin xyz="0.001 0 0" rpy=" 0 0 -1.5707"/>
-          <geometry>
-            <mesh filename="package://myrobot/models/myroboturdf/meshes/Boards/LattePanda_delta.dae" scale="0.001 0.001 0.001"/>
+          <origin xyz="0.001 0 0" rpy="1.5707 0 0 "/>
+          <geometry>
+            <mesh filename="package://myrobot/models/myroboturdf/meshes/Boards/LattePanda_delta.dae"/>
           </geometry>
       </visual>
@@ -605,5 +626,5 @@
       <parent link="BaseBoards"/>
       <child link="K64F"/>
-      <origin xyz="0 0 0.138" rpy="3.1415 0 1.5707"/>
+      <origin xyz="0 0 -0.003" rpy="3.1415 0 1.5707"/>
     </joint>
     <link name="K64F">
@@ -620,8 +641,13 @@
           </geometry>
       </collision>
+      <!-- <visual name="visual">
+          <geometry>
+            <box size="0.085 0.055 0.015"/>
+          </geometry>
+      </visual>   -->
       <visual name="visual">
           <origin xyz="-0.037 -0.027 -0.007" rpy=" 0 0 0"/>
           <geometry>
-            <mesh filename="package://myrobot/models/myroboturdf/meshes/Boards/K64F.dae" scale="0.001 0.001 0.001"/>
+            <mesh filename="package://myrobot/models/myroboturdf/meshes/Boards/K64F.dae"/>
           </geometry>
       </visual>
@@ -630,5 +656,5 @@
       <parent link="supporto_sg90"/>
       <child link="sg90h"/>
-      <origin xyz="0.106 -0.005 0.092" rpy="1.5707 0 0"/>
+      <origin xyz="0.003 -0.00 -0.01" rpy="1.5707 0 0"/>
     </joint>
     <link name="sg90h">
@@ -645,8 +671,13 @@
           </geometry>
       </collision>
+      <visual name="collision_sg90h">
+          <geometry>
+            <box size=".012 0.022 0.022"/>
+          </geometry>
+      </visual>
       <visual name="visual">
           <origin xyz="0 -0.011 0" rpy=" 0 0 0"/>
           <geometry>
-            <mesh filename="package://myrobot/models/myroboturdf/meshes/Misc/sg90.dae" scale="0.001 0.001 0.001"/>
+            <mesh filename="package://myrobot/models/myroboturdf/meshes/Misc/sg90.dae"/>
           </geometry>
       </visual>
@@ -655,5 +686,5 @@
       <parent link="sg90h"/>
       <child link="sg90h_shaft"/>
-      <origin xyz="0.106 0.0005 0.106" rpy="0 0 0"/>
+      <origin xyz="0.0 0 0.02" rpy="1.5707 0 0"/>
       <axis xyz="0 0 1"/>
     </joint>
@@ -677,5 +708,5 @@
       </visual>
     </link>
-    <joint name="sg90v_joint" type="fixed">
+    <!-- <joint name="sg90v_joint" type="fixed">
       <parent link="supporto_pitch_servo_2"/>
       <child link="sg90v"/>

Commit message: new additions and changes in the launch folder

File: models/myroboturdf/myrobot.gazebo.xacro (robot description, xacro)
@@ -73,4 +73,5 @@
   <gazebo reference="laser_sensor">
     <sensor type='ray' name='laser'>
+      <pose>0 0 0 0 0 0</pose>
       <visualize>true</visualize>
       <update_rate>5</update_rate>
@@ -162,11 +163,36 @@
     </plugin>
   </gazebo> -->
-  <!-- <gazebo>
-    <plugin name="gazebo_ros_lds_lfcd_controller" filename="libgazebo_ros_laser.so">
-      <topicName>scan</topicName>
-      <frameName>laser_scan</frameName>
-    </plugin>
-  </gazebo> -->
-  <gazebo>
+  <gazebo reference="laser_sensor">
+    <sensor type="ray" name="lds_lfcd_sensor">
+      <pose>0 0 0 0 0 0</pose>
+      <visualize>true</visualize>
+      <update_rate>5</update_rate>
+      <ray>
+        <scan>
+          <horizontal>
+            <samples>360</samples>
+            <resolution>1</resolution>
+            <min_angle>0.0</min_angle>
+            <max_angle>6.28319</max_angle>
+          </horizontal>
+        </scan>
+        <range>
+          <min>0.120</min>
+          <max>3.5</max>
+          <resolution>0.015</resolution>
+        </range>
+        <noise>
+          <type>gaussian</type>
+          <mean>0.0</mean>
+          <stddev>0.01</stddev>
+        </noise>
+      </ray>
+      <plugin name="gazebo_ros_lds_lfcd_controller" filename="libgazebo_ros_laser.so">
+        <topicName>scan</topicName>
+        <frameName>laser_sensor</frameName>
+      </plugin>
+    </sensor>
+  </gazebo>
+  <!-- <gazebo>
     <plugin name="cube_moving_code" filename="libdiff_drive_plugin.so">
         <commandTopic>cmd_vel</commandTopic>
@@ -189,5 +215,5 @@
         <rosDebugLevel>na</rosDebugLevel>
     </plugin>
-  </gazebo>
+  </gazebo> -->
   <!--<gazebo>
      <plugin name="ActuatorPlugin_horizontal" filename="libactuator_plugin.so">

File: models/myroboturdf/myrobot.urdf.xacro (robot description, xacro)
@@ -82,9 +82,9 @@
       </visual>
     </link>
-    <joint name="wheel_left_joint" type="continuous">
+    <joint name="left_wheel_hinge" type="continuous">
       <parent link="cube_base"/>
       <child link="wheel_left_link"/>
       <origin xyz="0. 0.087 -0.011" rpy="0 1.5707 1.5707"/>
-      <axis xyz="1 0 0"/>
+      <axis xyz=" 0 0 1"/>
     </joint>
     <link name="wheel_left_link">
@@ -107,9 +107,9 @@
       </visual>
     </link>
-    <joint name="wheel_right_joint" type="continuous">
+    <joint name="rigth_wheel_hinge" type="continuous">
       <parent link="cube_base"/>
       <child link="wheel_right_link"/>
       <origin xyz="0. -0.087 -0.011" rpy="0 0 0"/>
-      <axis xyz="1 0 0"/>
+      <axis xyz="0 1 0"/>
     </joint>
     <link name="wheel_right_link">
@@ -155,10 +155,10 @@
         </geometry>
       </visual>
-       <visual>
+       <!-- <visual>
         <origin xyz="0 0 0" rpy="0 0 0"/>
         <geometry>
           <box size="0.16 0.122315 0.002"/>
         </geometry>
-      </visual>
+      </visual> -->
       <collision name = "stick1_collision">
       <origin xyz="0.075 0.05 -0.02 " rpy="0 0 0"/>
@@ -270,8 +270,8 @@
       </visual> -->
     </link>
-    <!-- <joint name="supporto_piastra_albero_joint" type="fixed">
+    <joint name="supporto_piastra_albero_joint" type="fixed">
       <parent link="sg90h_shaft"/>
       <child link="supporto_piastra_albero"/>
-      <origin xyz="0.106 0.0005 0.109" rpy="0 0 0"/>
+      <origin xyz="0 0 -0.005" rpy="0 0 0"/>
     </joint>
     <link name="supporto_piastra_albero">
@@ -287,4 +287,10 @@
         </geometry>
       </collision>
+      <!-- <visual>
+        <origin xyz="0 0 0 " rpy="0 0 0"/>
+        <geometry>
+          <cylinder length="0.004" radius="0.008"/>
+        </geometry>
+      </visual> -->
       <visual>
         <origin xyz="0 0 -0.002" rpy="1.5707 0 4.71238"/>
@@ -293,5 +299,5 @@
         </geometry>
       </visual>
-    </link> -->
+    </link>
     <!-- <joint name="supporto_pitch_servo_1_joint" type="fixed">
       <parent link="supporto_piastra_albero"/>
@@ -686,5 +692,5 @@
       <parent link="sg90h"/>
       <child link="sg90h_shaft"/>
-      <origin xyz="0.0 0 0.02" rpy="1.5707 0 0"/>
+      <origin xyz="-0.0 0.015 -0.005" rpy="1.5707 0 0"/>
       <axis xyz="0 0 1"/>
     </joint>
