Commit message: checked tags in model and copied inside urdf

File: models/myroboturdf/myrobot.gazebo.xacro (robot description, xacro)
@@ -20,4 +20,26 @@
     <maxVel>0.1</maxVel>
     <fdir1>1 0 0</fdir1>
+  </gazebo>
+   <gazebo>
+    <plugin name="cube_moving_code" filename="libdiff_drive_plugin.so">
+        <commandTopic>cmd_vel</commandTopic>
+        <odometryTopic>odom</odometryTopic>
+        <odometryFrame>odom</odometryFrame>
+        <odometrySource>world</odometrySource>
+        <publishOdomTF>true</publishOdomTF>
+        <robotBaseFrame>base_footprint</robotBaseFrame>
+        <publishWheelTF>false</publishWheelTF>
+        <publishTf>true</publishTf>
+        <publishWheelJointState>true</publishWheelJointState>
+        <legacyMode>false</legacyMode>
+        <updateRate>30</updateRate>
+        <leftJoint>left_wheel_hinge</leftJoint>
+        <rightJoint>right_wheel_hinge</rightJoint>
+        <wheelSeparation>0.4</wheelSeparation>
+        <wheelDiameter>0.2</wheelDiameter>
+        <wheelAcceleration>1</wheelAcceleration>
+        <wheelTorque>10</wheelTorque>
+        <rosDebugLevel>na</rosDebugLevel>
+    </plugin>
   </gazebo>
   <!-- <gazebo reference="RealSense">
@@ -194,26 +216,4 @@
     </sensor>
   </gazebo>
-  <!-- <gazebo>
-    <plugin name="cube_moving_code" filename="libdiff_drive_plugin.so">
-        <commandTopic>cmd_vel</commandTopic>
-        <odometryTopic>odom</odometryTopic>
-        <odometryFrame>odom</odometryFrame>
-        <odometrySource>world</odometrySource>
-        <publishOdomTF>true</publishOdomTF>
-        <robotBaseFrame>base_footprint</robotBaseFrame>
-        <publishWheelTF>false</publishWheelTF>
-        <publishTf>true</publishTf>
-        <publishWheelJointState>true</publishWheelJointState>
-        <legacyMode>false</legacyMode>
-        <updateRate>30</updateRate>
-        <leftJoint>left_wheel_hinge</leftJoint>
-        <rightJoint>right_wheel_hinge</rightJoint>
-        <wheelSeparation>0.4</wheelSeparation>
-        <wheelDiameter>0.2</wheelDiameter>
-        <wheelAcceleration>1</wheelAcceleration>
-        <wheelTorque>10</wheelTorque>
-        <rosDebugLevel>na</rosDebugLevel>
-    </plugin>
-  </gazebo> -->
   <!--<gazebo>
      <plugin name="ActuatorPlugin_horizontal" filename="libactuator_plugin.so">

File: models/myroboturdf/myrobot.urdf.xacro (robot description, xacro)
@@ -20,5 +20,5 @@
                  izz="2.0064271e-03" />
       </inertial>
-      <collision name="collision_cube_base">
+      <collision name="cube_base_collision">
         <origin xyz="0 0 0 " rpy="0 0 0"/>
         <geometry>
@@ -26,5 +26,5 @@
         </geometry>
       </collision>
-     <visual name="visual">
+     <visual name="cube_base_visual">
         <geometry>
           <box size="0.19 0.134 0.047"/>
@@ -53,5 +53,5 @@
         </surface>
       </collision>
-      <visual name="caster_collision">
+      <visual name="caster_visual">
       <origin xyz="-0.05 0 -0.03" rpy="0 0 0"/>
         <geometry>
@@ -59,5 +59,5 @@
         </geometry>
       </visual>
-      <collision name = 'caster_collision2'>
+      <collision name = 'caster2_collision'>
       <origin xyz="0.05 0 -0.03" rpy="0 0 0"/>
         <geometry>
@@ -75,5 +75,5 @@
         </surface>
       </collision>
-      <visual name="caster_collision2">
+      <visual name="caster2_visual">
       <origin xyz="0.05 0 -0.03" rpy="0 0 0"/>
         <geometry>
@@ -94,5 +94,5 @@
         <inertia ixx="0.00052666666" ixy="0" ixz="0" iyy="0.00052666666" iyz="0" izz="0.001"/>
       </inertial>
-      <collision>
+      <collision name="wheel_left_link_collision">
         <origin xyz="0 0 0" rpy="0 0 0"/>
         <geometry>
@@ -100,5 +100,5 @@
         </geometry>
       </collision>
-      <visual>
+      <visual name="wheel_left_link_visual">
         <origin xyz="0 0 0" rpy="0 0 0"/>
         <geometry>
@@ -119,5 +119,5 @@
         <inertia ixx="0.00052666666" ixy="0" ixz="0" iyy="0.00052666666" iyz="0" izz="0.001"/>
       </inertial>
-      <collision>
+      <collision name="wheel_right_link_collision">
         <origin xyz="0 0 0" rpy="0 0 0"/>
         <geometry>
@@ -125,5 +125,5 @@
         </geometry>
       </collision>
-      <visual>
+      <visual name="wheel_right_link_visual">
         <origin xyz="0 0 0" rpy="1.57 0 0"/>
         <geometry>
@@ -143,5 +143,5 @@
         <inertia ixx="0.00052666666" ixy="0" ixz="0" iyy="0.00052666666" iyz="0" izz="0.001"/>
       </inertial>
-      <collision name="collision_BaseBoards">
+      <collision name="BaseBoards_collision">
         <origin xyz="0 0 0 " rpy="0 0 0"/>
         <geometry>
@@ -149,5 +149,5 @@
         </geometry>
       </collision>
-      <!-- <visual>
+      <!-- <visual  name="BaseBoards_visual">
         <origin xyz="0.05 0 0" rpy="0 0 1.5707"/>
         <geometry>
@@ -155,5 +155,5 @@
         </geometry>
       </visual> -->
-       <visual>
+       <visual name="BaseBoards_visual">
         <origin xyz="0 0 0" rpy="0 0 0"/>
         <geometry>
@@ -167,5 +167,5 @@
         </geometry>
       </collision>
-      <visual name="stick1_collision">
+      <visual name="stick1_visual">
       <origin xyz="0.075 0.05 -0.02 " rpy="0 0 0"/>
         <geometry>
@@ -179,5 +179,5 @@
         </geometry>
       </collision>
-      <visual name="stick2_collision">
+      <visual name="stick2_visual">
       <origin xyz="0.075 -0.05 -0.02 " rpy="0 0 0"/>
         <geometry>
@@ -191,5 +191,5 @@
         </geometry>
       </collision>
-      <visual name="stick3_collision">
+      <visual name="stick3_visual">
       <origin xyz="-0.075 -0.05 -0.02 " rpy="0 0 0"/>
         <geometry>
@@ -203,5 +203,5 @@
         </geometry>
       </collision>
-      <visual name="stick4_collision">
+      <visual name="stick4_visual">
       <origin xyz="-0.075 0.05 -0.02 " rpy="0 0 0"/>
         <geometry>
@@ -221,5 +221,5 @@
         <inertia ixx="0.00052666666" ixy="0" ixz="0" iyy="0.00052666666" iyz="0" izz="0.001"/>
       </inertial>
-      <collision name="collision_piastra_anteriore">
+      <collision name="piastra_anteriore_collision">
         <origin xyz="0 0 0 " rpy="0 0 0"/>
         <geometry>
@@ -227,5 +227,5 @@
         </geometry>
       </collision>
-      <visual>
+      <visual name ="piastra_anteriore_visual">
         <origin xyz="0 0 0 " rpy="0 0 0"/>
         <geometry>
@@ -251,5 +251,5 @@
         <inertia ixx="0.00052666666" ixy="0" ixz="0" iyy="0.00052666666" iyz="0" izz="0.001"/>
       </inertial>
-      <collision name="collision_supporto_sg90">
+      <collision name="supporto_sg90_collision">
         <origin xyz="0 0 0 " rpy="0 0 0"/>
         <geometry>
@@ -263,5 +263,5 @@
         </geometry>
       </visual> -->
-      <visual>
+      <visual name="supporto_sg90_visual">
         <origin xyz="0 0 0 " rpy="0 0 0"/>
         <geometry>
@@ -281,5 +281,5 @@
         <inertia ixx="0.00052666666" ixy="0" ixz="0" iyy="0.00052666666" iyz="0" izz="0.001"/>
       </inertial>
-      <collision name="collision_supporto_sg90">
+      <collision name="supporto_piastra_albero_collision">
         <origin xyz="0 0 0 " rpy="0 0 0"/>
         <geometry>
@@ -287,5 +287,5 @@
         </geometry>
       </collision>
-      <visual>
+      <visual name="supporto_piastra_albero_visual">
         <origin xyz="0 0 0 " rpy="0 0 0"/>
         <geometry>
@@ -293,5 +293,5 @@
         </geometry>
       </visual>
-      <!-- <visual>
+      <!-- <visual name="supporto_piastra_albero_visual">
         <origin xyz="0 0 -0.002" rpy="1.5707 0 4.71238"/>
         <geometry>
@@ -316,5 +316,5 @@
         </inertia>
       </inertial>
-      <collision name='collision'>
+      <collision name='supporto_pitch_servo_1_collision'>
         <geometry>
           <box>
@@ -323,5 +323,5 @@
         </geometry>
       </collision>
-      <visual name='visual'>
+      <visual name='supporto_pitch_servo_1_visual'>
       <pose>0.0375 0 -0.003 0 0 0</pose>
         <geometry>
@@ -335,5 +335,5 @@
         </material>
       </visual>
-      <collision name='collision_tronco1'>
+      <collision name='tronco1_collision'>
       <pose>0.0 0.0 -0.001 0 0 0</pose>
         <geometry>
@@ -349,5 +349,5 @@
         </geometry>
       </collision>
-      <collision name='collision_cube2'>
+      <collision name='cube2_collision'>
       <pose>0.076 0 0 0 0 0</pose>
         <geometry>
@@ -357,5 +357,5 @@
         </geometry>
       </collision>
-      <collision name='collision_cil'>
+      <collision name='cil_collision'>
       <pose>0.038 0.0 0 0 0 0</pose>
         <geometry>
@@ -385,5 +385,5 @@
         </inertia>
       </inertial>
-      <collision name='collision'>
+      <collision name='supporto_pitch_servo_2_collision'>
         <geometry>
           <box>
@@ -392,5 +392,5 @@
         </geometry>
       </collision>
-      <visual name='visual'>
+      <visual name='supporto_pitch_servo_2_visual'>
       <pose>0.039 0 -0.001 0 0 0</pose>
         <geometry>
@@ -404,5 +404,5 @@
         </material>
       </visual>
-      <collision name='collision_vertical'>
+      <collision name='vertical_collision'>
       <pose>-0.002375 0 0.018 0 0 0 </pose>
         <geometry>
@@ -430,5 +430,5 @@
         </inertia>
       </inertial>
-      <collision name='collision'>
+      <collision name='supporto_pitch_servo_2_noservo_collision'>
         <geometry>
           <box>
@@ -437,5 +437,5 @@
         </geometry>
       </collision>
-      <visual name='visual'>
+      <visual name='supporto_pitch_servo_2_noservo_visual'>
       <pose>0.082 0 -0.001 0 0 3.1415</pose>
         <geometry>
@@ -449,5 +449,5 @@
         </material>
       </visual>
-      <collision name='collision_vertical'>
+      <collision name='vertical2_collision'>
       <pose>-0.002375 0 0.018 0 0 0 </pose>
         <geometry>
@@ -473,5 +473,5 @@
         </geometry>
       </collision>
-     <visual name='visual'>
+     <visual name='supp_RS_visual'>
       <pose>0.0 0.054 0.013 1.5707 0 1.5707</pose>
         <geometry>
@@ -485,5 +485,5 @@
         </material>
       </visual>
-      <collision name='collision_vertical'>
+      <collision name='vertical3_collision'>
       <pose>0 0.05 0.01 0 0 0 </pose>
         <geometry>
@@ -493,5 +493,5 @@
         </geometry>
       </collision>
-      <collision name='collision_vertical2'>
+      <collision name='vertical4_collision'>
       <pose>0 -0.05 0.01 0 0 0 </pose>
         <geometry>
@@ -509,10 +509,10 @@
     </joint>
     <link name="RealSense">
-        <collision name="collision">
+        <collision name="RealSense_collision">
           <geometry>
             <box size="0.025 0.087 0.02"/>
           </geometry>
         </collision>
-        <visual name="visual">
+        <visual name="RealSense_visual">
           <origin xyz="0.0125 0.0 0" rpy="1.5707 0 1.5707"/>
           <geometry>
@@ -527,10 +527,10 @@
     </joint>
     <link name="rightfront_force_sensor">
-        <visual name="visual">
+        <visual name="rightfront_force_sensor_visual">
           <geometry>
             <box size="0.05 0.01 0.01"/>
           </geometry>
         </visual>
-        <collision name="collision_rightfront_collision">
+        <collision name="rightfront_force_sensor_collision">
           <geometry>
             <box size="0.05 0.01 0.01"/>
@@ -544,10 +544,10 @@
     </joint>
     <link name="leftfront_force_sensor">
-        <visual name="visual">
+        <visual name="leftfront_force_sensor_visual">
           <geometry>
             <box size="0.05 0.01 0.01"/>
           </geometry>
         </visual>
-        <collision name="collision_leftfront_collision">
+        <collision name="leftfront_force_sensor_collision">
           <geometry>
             <box size="0.05 0.01 0.01"/>
@@ -568,5 +568,5 @@
                    izz="2.0712558e-05" />
         </inertial>
-        <!-- <visual name="visual">
+        <!-- <visual name="LightSensor_visual">
           <origin xyz="0.001 0 0" rpy=" 0 0 -1.5707"/>
           <geometry>
@@ -574,5 +574,5 @@
           </geometry>
         </visual> -->
-        <visual name="visual">
+        <visual name="LightSensor_visual">
           <origin xyz="0.001 0 0" rpy=" 0 0 -1.5707"/>
           <geometry>
@@ -580,5 +580,5 @@
           </geometry>
         </visual>
-        <collision name="collision">
+        <collision name="LightSensor_collision">
           <geometry>
             <box size="0.005 0.01 0.01"/>
@@ -599,5 +599,5 @@
                    izz="2.0712558e-05" />
         </inertial>
-        <collision name="collision_laser_sensor">
+        <collision name="laser_sensor_collision">
           <geometry>
             <box size="0.05 0.01 0.01"/>
@@ -618,15 +618,15 @@
                    izz="2.0712558e-05" />
       </inertial>
-      <collision name="collision_LattePanda">
+      <collision name="LattePanda_collision">
           <geometry>
             <box size="0.12 0.08 0.01"/>
           </geometry>
       </collision>
-      <visual name="visual">
+      <visual name="LattePanda_visual">
           <geometry>
             <box size="0.12 0.08 0.01"/>
           </geometry>
       </visual>
-      <!-- <visual name="visual">
+      <!-- <visual name="LattePanda_visual">
           <origin xyz="0.001 0 0" rpy="1.5707 0 0 "/>
           <geometry>
@@ -638,5 +638,5 @@
       <parent link="BaseBoards"/>
       <child link="K64F"/>
-      <origin xyz="0 0 -0.003" rpy="3.1415 0 1.5707"/>
+      <origin xyz="0 0 -0.0045" rpy="3.1415 0 1.5707"/>
     </joint>
     <link name="K64F">
@@ -648,10 +648,10 @@
                    izz="2.0712558e-05" />
       </inertial>
-      <collision name="collision_K64F">
+      <collision name="K64F_collision">
           <geometry>
             <box size="0.085 0.055 0.015"/>
           </geometry>
       </collision>
-      <visual name="visual">
+      <visual name="K64F_visual">
           <geometry>
             <box size="0.085 0.055 0.015"/>
@@ -678,15 +678,15 @@
                    izz="2.0712558e-05" />
       </inertial>
-      <collision name="collision_sg90h">
+      <collision name="sg90h_collision">
           <geometry>
             <box size=".012 0.022 0.022"/>
           </geometry>
       </collision>
-      <visual name="collision_sg90h">
+      <visual name="sg90h_visual">
           <geometry>
             <box size=".012 0.022 0.022"/>
           </geometry>
       </visual>
-      <!-- <visual name="visual">
+      <!-- <visual name="sg90h_visual">
           <origin xyz="0 -0.011 0" rpy=" 0 0 0"/>
           <geometry>
@@ -709,10 +709,10 @@
                    izz="2.0712558e-05" />
       </inertial>
-      <collision name="collision_sg90h_shaft">
+      <collision name="sg90h_shaft_collision">
         <geometry>
           <cylinder length="0.01" radius="0.002"/>
         </geometry>
       </collision>
-      <visual name="visual">
+      <visual name="sg90h_shaft_visual">
         <geometry>
           <cylinder length="0.01" radius="0.002"/>
@@ -733,10 +733,10 @@
                    izz="2.0712558e-05" />
       </inertial>
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
Commit message: working laser and diff drive

File: models/myroboturdf/myrobot.gazebo.xacro (robot description, xacro)
@@ -22,23 +22,23 @@
   </gazebo>
    <gazebo>
-    <plugin name="cube_moving_code" filename="libdiff_drive_plugin.so">
-        <commandTopic>cmd_vel</commandTopic>
-        <odometryTopic>odom</odometryTopic>
-        <odometryFrame>odom</odometryFrame>
-        <odometrySource>world</odometrySource>
-        <publishOdomTF>true</publishOdomTF>
-        <robotBaseFrame>base_footprint</robotBaseFrame>
-        <publishWheelTF>false</publishWheelTF>
-        <publishTf>true</publishTf>
-        <publishWheelJointState>true</publishWheelJointState>
-        <legacyMode>false</legacyMode>
-        <updateRate>30</updateRate>
-        <leftJoint>left_wheel_hinge</leftJoint>
-        <rightJoint>right_wheel_hinge</rightJoint>
-        <wheelSeparation>0.4</wheelSeparation>
-        <wheelDiameter>0.2</wheelDiameter>
-        <wheelAcceleration>1</wheelAcceleration>
-        <wheelTorque>10</wheelTorque>
-        <rosDebugLevel>na</rosDebugLevel>
+    <plugin name="turtlebot3_burger_controller" filename="libdiff_drive_plugin.so">
+      <commandTopic>cmd_vel</commandTopic>
+      <odometryTopic>odom</odometryTopic>
+      <odometryFrame>odom</odometryFrame>
+      <odometrySource>world</odometrySource>
+      <publishOdomTF>true</publishOdomTF>
+      <robotBaseFrame>base_footprint</robotBaseFrame>
+      <publishWheelTF>false</publishWheelTF>
+      <publishTf>true</publishTf>
+      <publishWheelJointState>true</publishWheelJointState>
+      <legacyMode>false</legacyMode>
+      <updateRate>30</updateRate>
+      <leftJoint>wheel_left_joint</leftJoint>
+      <rightJoint>wheel_right_joint</rightJoint>
+      <wheelSeparation>0.160</wheelSeparation>
+      <wheelDiameter>0.066</wheelDiameter>
+      <wheelAcceleration>1</wheelAcceleration>
+      <wheelTorque>10</wheelTorque>
+      <rosDebugLevel>na</rosDebugLevel>
     </plugin>
   </gazebo>
@@ -60,5 +60,5 @@
     </sensor>
   </gazebo>-->
-  <gazebo reference="rightfront_force_sensor">
+  <!-- <gazebo reference="rightfront_force_sensor">
     <sensor name="rf_force_sensor" type="contact">
       <update_rate>30.0</update_rate>
@@ -77,6 +77,6 @@
       </contact>
     </sensor>
-  </gazebo>
-<gazebo reference="LightSensor">
+  </gazebo> -->
+<!-- <gazebo reference="LightSensor">
     <sensor name='camera' type='depth'>
       <camera name='camera'>
@@ -92,32 +92,5 @@
       </camera>
     </sensor>
-  </gazebo>
-  <gazebo reference="laser_sensor">
-    <sensor type='ray' name='laser'>
-      <pose>0 0 0 0 0 0</pose>
-      <visualize>true</visualize>
-      <update_rate>5</update_rate>
-      <ray>
-        <scan>
-          <horizontal>
-            <samples>360</samples>
-            <resolution>1</resolution>
-            <min_angle>0.0</min_angle>
-            <max_angle>6.28319</max_angle>
-          </horizontal>
-        </scan>
-        <range>
-          <min>0.120</min>
-          <max>3.5</max>
-          <resolution>0.015</resolution>
-        </range>
-        <noise>
-          <type>gaussian</type>
-          <mean>0.0</mean>
-          <stddev>0.01</stddev>
-        </noise>
-      </ray>
-    </sensor>
-  </gazebo>
+  </gazebo> -->
 <!-- PLUGINS -->
   <!-- <gazebo>

File: models/myroboturdf/myrobot.urdf.xacro (robot description, xacro)
@@ -2,7 +2,5 @@
 <robot name="myrobot" xmlns:xacro="http://ros.org/wiki/xacro">
   <xacro:include filename="$(find myrobot)/models/myroboturdf/myrobot.gazebo.xacro"/>
-    <!-- <static>false</static>
-    <self_collide>false</self_collide> -->
-    <!-- LINKS -->
+<!-- LINKS -->
     <link name="base_footprint"/>
     <joint name="base_joint" type="fixed">
@@ -11,5 +9,4 @@
       <origin xyz="0.0 0.0 0.08" rpy="0 0 0"/>
     </joint>
-    <!--%%%%%%%%%%%%%%%%%%%%%%%%%%%%%%%%%%%%%%%%%BODY%%%%%%%%%%%%%%%%%%%%%%%%%%%%%%%%%%%%%%%%%%%%%%-->
     <link name="cube_base">
       <inertial>
@@ -82,9 +79,9 @@
       </visual>
     </link>
-    <joint name="left_wheel_hinge" type="continuous">
+    <joint name="wheel_left_joint" type="continuous">
       <parent link="cube_base"/>
       <child link="wheel_left_link"/>
-      <origin xyz="0. 0.087 -0.011" rpy="0 1.5707 1.5707"/>
-      <axis xyz=" 0 0 1"/>
+      <origin xyz="0. 0.087 -0.014" rpy="-1.57 0 0"/>
+      <axis xyz="0 0 1"/>
     </joint>
     <link name="wheel_left_link">
@@ -95,5 +92,5 @@
       </inertial>
       <collision name="wheel_left_link_collision">
-        <origin xyz="0 0 0" rpy="0 0 0"/>
+        <!-- <origin xyz="0 0 0" rpy="0 0 0"/> -->
         <geometry>
           <cylinder length="0.035" radius="0.06825"/>
@@ -107,9 +104,9 @@
       </visual>
     </link>
-    <joint name="rigth_wheel_hinge" type="continuous">
+    <joint name="wheel_right_joint" type="continuous">
       <parent link="cube_base"/>
       <child link="wheel_right_link"/>
-      <origin xyz="0. -0.087 -0.011" rpy="0 0 0"/>
-      <axis xyz="0 1 0"/>
+      <origin xyz="0. -0.087 -0.014" rpy="-1.57 0 0"/>
+      <axis xyz="0 0 1"/>
     </joint>
     <link name="wheel_right_link">
@@ -120,11 +117,11 @@
       </inertial>
       <collision name="wheel_right_link_collision">
+        <!-- <origin xyz="0 0 0" rpy="0 0 0"/> -->
+        <geometry>
+          <cylinder length="0.035" radius="0.06825"/>
+        </geometry>
+      </collision>
+      <visual name="wheel_right_link_visual">
         <origin xyz="0 0 0" rpy="0 0 0"/>
-        <geometry>
-          <cylinder length="0.035" radius="0.06825"/>
-        </geometry>
-      </collision>
-      <visual name="wheel_right_link_visual">
-        <origin xyz="0 0 0" rpy="1.57 0 0"/>
         <geometry>
           <cylinder length="0.035" radius="0.06825"/>
