Commit message: removed most of inertias. Sensitive

File: models/myroboturdf/myrobot.gazebo.xacro (robot description, xacro)
@@ -9,5 +9,5 @@
     <kd>10.0</kd>
     <minDepth>0.001</minDepth>
-    <maxVel>0.1</maxVel>
+    <maxVel>1</maxVel>
     <fdir1>1 0 0</fdir1>
   </gazebo>
@@ -18,5 +18,5 @@
     <kd>10.0</kd>
     <minDepth>0.001</minDepth>
-    <maxVel>0.1</maxVel>
+    <maxVel>1</maxVel>
     <fdir1>1 0 0</fdir1>
   </gazebo>
@@ -161,5 +161,5 @@
     <sensor type="ray" name="lds_lfcd_sensor">
       <pose>0 0 0 0 0 0</pose>
-      <visualize>true</visualize>
+      <visualize>false</visualize>
       <update_rate>5</update_rate>
       <ray>

File: models/myroboturdf/myrobot.urdf.xacro (robot description, xacro)
@@ -12,5 +12,5 @@
       <inertial>
         <origin xyz="0 0 0" rpy="0 0 0"/>
-        <mass value="8.2573504e-01"/>
+        <mass value="0.2"/>
         <inertia ixx="2.2124416e-03" ixy="-1.2294101e-05" ixz="3.4938785e-05"
                  iyy="2.1193702e-03" iyz="-5.0120904e-06"
@@ -82,5 +82,5 @@
       <parent link="cube_base"/>
       <child link="wheel_left_link"/>
-      <origin xyz="0. 0.087 -0.014" rpy="-1.57 0 0"/>
+      <origin xyz="0. 0.087 -0.021" rpy="-1.57 0 0"/>
       <axis xyz="0 0 1"/>
     </joint>
@@ -94,5 +94,5 @@
         <!-- <origin xyz="0 0 0" rpy="0 0 0"/> -->
         <geometry>
-          <cylinder length="0.035" radius="0.06825"/>
+          <cylinder length="0.035" radius="0.06"/>
         </geometry>
       </collision>
@@ -100,5 +100,5 @@
         <origin xyz="0 0 0" rpy="0 0 0"/>
         <geometry>
-          <cylinder length="0.035" radius="0.06825"/>
+          <cylinder length="0.035" radius="0.06"/>
         </geometry>
       </visual>
@@ -107,5 +107,5 @@
       <parent link="cube_base"/>
       <child link="wheel_right_link"/>
-      <origin xyz="0. -0.087 -0.014" rpy="-1.57 0 0"/>
+      <origin xyz="0. -0.087 -0.021" rpy="-1.57 0 0"/>
       <axis xyz="0 0 1"/>
     </joint>
@@ -119,5 +119,5 @@
         <!-- <origin xyz="0 0 0" rpy="0 0 0"/> -->
         <geometry>
-          <cylinder length="0.035" radius="0.06825"/>
+          <cylinder length="0.035" radius="0.06"/>
         </geometry>
       </collision>
@@ -125,5 +125,5 @@
         <origin xyz="0 0 0" rpy="0 0 0"/>
         <geometry>
-          <cylinder length="0.035" radius="0.06825"/>
+          <cylinder length="0.035" radius="0.06"/>
         </geometry>
       </visual>
@@ -135,9 +135,4 @@
     </joint>
     <link name="BaseBoards">
-      <inertial>
-        <mass value="0.2"/>
-        <origin rpy="0 0 0" xyz="0 0 0"/>
-        <inertia ixx="0.00052666666" ixy="0" ixz="0" iyy="0.00052666666" iyz="0" izz="0.001"/>
-      </inertial>
       <collision name="BaseBoards_collision">
         <origin xyz="0 0 0 " rpy="0 0 0"/>
@@ -213,9 +208,4 @@
     </joint>
     <link name="piastra_anteriore">
-      <inertial>
-        <mass value="0.2"/>
-        <origin rpy="0.078 -0.004 0.104" xyz="0 0 0"/>
-        <inertia ixx="0.00052666666" ixy="0" ixz="0" iyy="0.00052666666" iyz="0" izz="0.001"/>
-      </inertial>
       <collision name="piastra_anteriore_collision">
         <origin xyz="0 0 0 " rpy="0 0 0"/>
@@ -243,9 +233,4 @@
     </joint>
     <link name="supporto_sg90">
-      <inertial>
-        <mass value="0.2"/>
-        <origin rpy="0.078 -0.004 0.104" xyz="0 0 0"/>
-        <inertia ixx="0.00052666666" ixy="0" ixz="0" iyy="0.00052666666" iyz="0" izz="0.001"/>
-      </inertial>
       <collision name="supporto_sg90_collision">
         <origin xyz="0 0 0 " rpy="0 0 0"/>
@@ -558,5 +543,5 @@
     </joint>
     <link name="LightSensor">
-        <inertial>
+        <!-- <inertial>
           <origin xyz="0 0 0" />
           <mass value="2.8498940e-02" />
@@ -564,5 +549,5 @@
                    iyy="1.1192413e-05" iyz="-1.4400107e-11"
                    izz="2.0712558e-05" />
-        </inertial>
+        </inertial> -->
         <!-- <visual name="LightSensor_visual">
           <origin xyz="0.001 0 0" rpy=" 0 0 -1.5707"/>
@@ -608,11 +593,4 @@
     </joint>
     <link name="LattePanda">
-      <inertial>
-          <origin xyz="0 0 0" />
-          <mass value="2.8498940e-02" />
-          <inertia ixx="1.1175580e-05" ixy="-4.2369783e-11" ixz="-5.9381719e-09"
-                   iyy="1.1192413e-05" iyz="-1.4400107e-11"
-                   izz="2.0712558e-05" />
-      </inertial>
       <collision name="LattePanda_collision">
           <geometry>
@@ -638,11 +616,4 @@
     </joint>
     <link name="K64F">
-      <inertial>
-          <origin xyz="0 0 0" />
-          <mass value="2.8498940e-02" />
-          <inertia ixx="1.1175580e-05" ixy="-4.2369783e-11" ixz="-5.9381719e-09"
-                   iyy="1.1192413e-05" iyz="-1.4400107e-11"
-                   izz="2.0712558e-05" />
-      </inertial>
       <collision name="K64F_collision">
           <geometry>
@@ -668,5 +639,5 @@
     </joint>
     <link name="sg90h">
-      <inertial>
+      <!-- <inertial>
           <origin xyz="0 0 0" />
           <mass value="2.8498940e-02" />
@@ -674,5 +645,5 @@
                    iyy="1.1192413e-05" iyz="-1.4400107e-11"
                    izz="2.0712558e-05" />
-      </inertial>
+      </inertial> -->
       <collision name="sg90h_collision">
           <geometry>

Commit message: adding rest of parts. Actuator h works

File: models/myroboturdf/myrobot.gazebo.xacro (robot description, xacro)
@@ -2,4 +2,5 @@
 <robot name="myrobot_sim" xmlns:xacro="http://ros.org/wiki/xacro">
   <gazebo reference="cube_base">
+  <material>Gazebo/Grey</material>
   </gazebo>
   <gazebo reference="wheel_left_link">
@@ -11,4 +12,5 @@
     <maxVel>1</maxVel>
     <fdir1>1 0 0</fdir1>
+    <material>light_black</material>
   </gazebo>
   <gazebo reference="wheel_right_link">
@@ -20,4 +22,5 @@
     <maxVel>1</maxVel>
     <fdir1>1 0 0</fdir1>
+    <material>Gazebo/FlatBlack</material>
   </gazebo>
    <gazebo>
@@ -42,4 +45,10 @@
       <rosDebugLevel>na</rosDebugLevel>
     </plugin>
+  </gazebo>
+  <gazebo reference="sg90h_shaft">
+    <material>Gazebo/Red</material>
+  </gazebo>
+  <gazebo reference="supporto_pitch_servo_1">
+    <!-- <material>Gazebo/Blue</material> -->
   </gazebo>
   <!-- <gazebo reference="RealSense">
@@ -189,7 +198,7 @@
     </sensor>
   </gazebo>
-  <!--<gazebo>
+  <gazebo>
      <plugin name="ActuatorPlugin_horizontal" filename="libactuator_plugin.so">
-        <motor_joint>sg90h_to_shaft</motor_joint>
+        <motor_joint>sg90h_shaft_joint</motor_joint>
         <commandTopicServo>cmd_servo</commandTopicServo>
         <servoTorque>10</servoTorque>
@@ -201,5 +210,5 @@
         <robotNamespace>sg90h</robotNamespace>
         <servoodometrySource>world</servoodometrySource>
-        <servoBaseFrame>sg90h</servoBaseFrame>
+        <servoBaseFrame>supporto_sg90</servoBaseFrame>
         <publishServoTF>true</publishServoTF>
         <publishTF>true</publishTF>
@@ -207,5 +216,5 @@
         <rosDebugLevel>na</rosDebugLevel>
       </plugin>
-  </gazebo>-->
+  </gazebo>
  <!--  <gazebo>
     <plugin name="ActuatorPlugin_vertical" filename="libactuator_plugin.so">

File: models/myroboturdf/myrobot.urdf.xacro (robot description, xacro)
@@ -2,4 +2,5 @@
 <robot name="myrobot" xmlns:xacro="http://ros.org/wiki/xacro">
   <xacro:include filename="$(find myrobot)/models/myroboturdf/myrobot.gazebo.xacro"/>
+  <xacro:include filename="$(find myrobot)/models/myroboturdf/common_properties.xacro"/>
 <!-- LINKS -->
     <link name="base_footprint"/>
@@ -33,4 +34,5 @@
           <mesh filename="package://myrobot/models/myroboturdf/meshes/Devastator.stl" scale="0.001 0.001 0.001"/>
         </geometry>
+        <material name="light_black"/> <!--rviz colour-->
       </visual>
       <collision name = "caster_collision">
@@ -221,5 +223,5 @@
         <origin xyz="0.025 0 -0.0015 " rpy="0 0 1.5707"/>
         <geometry>
-          <mesh filename="package://myrobot/models/myroboturdf/meshes/Supports/Piastra_anteriore2.stl"/>
+          <mesh filename="package://myrobot/models/myroboturdf/meshes/Supports/Piastra_anteriore2.stl" scale="0.001 0.001 0.001"/>
         </geometry>
       </visual>
@@ -237,18 +239,18 @@
         </geometry>
       </collision>
-      <!-- <visual>
+      <visual>
         <origin xyz="-0.003 0.015 0" rpy="0 0 1.5707"/>
         <geometry>
-          <mesh filename="package://myrobot/models/myroboturdf/meshes/Supports/Supporto_sg90_base.dae"/>
-        </geometry>
-      </visual> -->
-      <visual name="supporto_sg90_visual">
+          <mesh filename="package://myrobot/models/myroboturdf/meshes/Supports/Supporto_sg90_base.stl" scale="0.001 0.001 0.001"/>
+        </geometry>
+      </visual>
+      <!-- <visual name="supporto_sg90_visual">
         <origin xyz="0 0 0 " rpy="0 0 0"/>
         <geometry>
           <box size="0.027 0.049 0.004"/>
         </geometry>
-      </visual>
-    </link>
-   <!--  <joint name="supporto_piastra_albero_joint" type="fixed">
+      </visual> -->
+    </link>
+    <joint name="supporto_piastra_albero_joint" type="fixed">
       <parent link="sg90h_shaft"/>
       <child link="supporto_piastra_albero"/>
@@ -276,122 +278,54 @@
         <origin xyz="0 0 -0.002" rpy="1.5707 0 4.71238"/>
         <geometry>
-          <mesh filename="package://myrobot/models/myroboturdf/meshes/Supports/Supporto_piastra_albero.dae" scale="1 1 1"/>
-        </geometry>
-      </visual>
-    </link>-->
-    <!-- <joint name="supporto_pitch_servo_1_joint" type="fixed">
+          <mesh filename="package://myrobot/models/myroboturdf/meshes/Supports/Supporto_piastra_albero.stl" scale="0.001 0.001 0.001"/>
+        </geometry>
+      </visual>
+    </link>
+    <joint name="supporto_pitch_servo_1_joint" type="fixed">
       <parent link="supporto_piastra_albero"/>
       <child link="supporto_pitch_servo_1"/>
-      <origin xyz="0.106 0.038 0.114" rpy="0 0 4.71238"/>
-    </joint>
-    <gazebo>
+      <origin xyz="0 0 -0.004" rpy="0 0 0" />
+    </joint>
     <link name='supporto_pitch_servo_1'>
-      <inertial>
-        <mass>0.1</mass>
-        <origin xyz="0.0 0 0" rpy=" 0 0 0"/>
-        <inertia>
-          <ixx>0.001</ixx> <ixy>0</ixy> <ixz>0</ixz>
-          <iyy>0.001</iyy> <iyz>0</iyz>
-          <izz>0.001</izz>
-        </inertia>
-      </inertial>
       <collision name='supporto_pitch_servo_1_collision'>
         <geometry>
-          <box>
-            <size>0.043 0.035 0.003</size>
-          </box>
-        </geometry>
-      </collision>
+          <box size="0.035 0.12 0.003"/>
+        </geometry>
+      </collision>
+      <!-- <visual name="supporto_pitch_servo_1_visual">
+        <geometry>
+          <box size="0.035 0.12 0.003"/>
+        </geometry>
+      </visual> -->
       <visual name='supporto_pitch_servo_1_visual'>
-      <pose>0.0375 0 -0.003 0 0 0</pose>
-        <geometry>
-          <mesh><uri>model://myrobot/meshes/Supports/supporto_pitch_servo_1_new.dae</uri></mesh>
-        </geometry>
-        <material>
-          <ambient>0 0 0.196 0.490</ambient>
-          <diffuse>0.043 0.043 0.043 1</diffuse>
-          <specular>.027 .027 .459 64</specular>
-          <emissive>0.047 0.035 0.286 1</emissive>
-        </material>
-      </visual>
-      <collision name='tronco1_collision'>
-      <pose>0.0 0.0 -0.001 0 0 0</pose>
-        <geometry>
-          <polyline>
-            <point> 0.02 -0.0175</point>
-            <point>0.0375 -0.008</point>
-            <point>0.055 -0.0175</point>
-            <point>0.055 0.0175</point>
-            <point>0.0375 0.008</point>
-            <point> 0.02 0.0175</point>
-            <height>0.003</height>
-          </polyline>
-        </geometry>
-      </collision>
-      <collision name='cube2_collision'>
-      <pose>0.076 0 0 0 0 0</pose>
-        <geometry>
-          <box>
-            <size>0.043 0.035 0.003</size>
-          </box>
-        </geometry>
-      </collision>
-      <collision name='cil_collision'>
-      <pose>0.038 0.0 0 0 0 0</pose>
-        <geometry>
-          <cylinder>
-            <radius>0.0075</radius>
-            <length>0.003</length>
-          </cylinder>
-        </geometry>
-      </collision>
-    </link>
-    </gazebo> -->
-    <!-- <joint name="supporto_pitch_servo_2_joint" type="fixed">
+      <origin xyz="0 0 0.004" rpy="3.1415 0 1.5707" />
+        <geometry>
+          <mesh filename="package://myrobot/models/myroboturdf/meshes/Supports/supporto_pitch_servo_1_new.stl" scale="0.001 0.001 0.001"/>
+        </geometry>
+      </visual>
+    </link>
+    <joint name="supporto_pitch_servo_2_joint" type="fixed">
       <parent link="supporto_pitch_servo_1"/>
       <child link="supporto_pitch_servo_2"/>
-      <origin xyz="0.106 0.056 0.116" rpy="0 0 4.71238"/>
-    </joint>
-    <gazebo>
+      <origin xyz="0.1 0 0" rpy="0 0 0"/>
+    </joint>
     <link name='supporto_pitch_servo_2'>
-    <self_collide>true</self_collide>
-      <inertial>
-        <mass>0.1</mass>
-        <origin xyz="0.0 0 0" rpy=" 0 0 0"/>
-        <inertia>
-          <ixx>0.001</ixx> <ixy>0</ixy> <ixz>0</ixz>
-          <iyy>0.001</iyy> <iyz>0</iyz>
-          <izz>0.001</izz>
-        </inertia>
-      </inertial>
       <collision name='supporto_pitch_servo_2_collision'>
         <geometry>
-          <box>
-            <size>0.0075 0.035 0.002</size>
-          </box>
+          <box size="0.002 0.02 0.035"/>
         </geometry>
       </collision>
       <visual name='supporto_pitch_servo_2_visual'>
-      <pose>0.039 0 -0.001 0 0 0</pose>
-        <geometry>
-          <mesh><uri>model://myrobot/meshes/Supports/supporto_pitch_servo_2.dae</uri></mesh>
-        </geometry>
-        <material>
-          <ambient>0 0 0.196 0.490</ambient>
-          <diffuse>0.043 0.043 0.043 1</diffuse>
-          <specular>.027 .027 .459 64</specular>
-          <emissive>0.047 0.035 0.286 1</emissive>
-        </material>
-      </visual>
-      <collision name='vertical_collision'>
-      <pose>-0.002375 0 0.018 0 0 0 </pose>
-        <geometry>
-          <box>
-            <size>0.002 0.02 0.035</size>
-          </box>
-        </geometry>
-      </collision>
-    </link>
-    </gazebo> -->
+      <origin xyz="0 0 0.02" rpy="0 3.1415 0" />
+        <geometry>
+          <mesh filename="package://myrobot/models/myroboturdf/meshes/Supports/supporto_pitch_servo_2.stl" scale="0.001 0.001 0.001"/>
+        </geometry>
+      </visual>
+      <visual name='supporto_pitch_servo_2_visual'>
+        <geometry>
+          <box size="0.002 0.02 0.035"/>
+        </geometry>
+      </visual>
+    </link>
     <!-- <joint name="supporto_pitch_servo_2_noservo_joint" type="fixed">
       <parent link="supporto_pitch_servo_1"/>
@@ -637,5 +571,5 @@
     </joint>
     <link name="sg90h">
-      <!-- <inertial>
+      <inertial>
           <origin xyz="0 0 0" />
           <mass value="2.8498940e-02" />
@@ -643,5 +577,5 @@
                    iyy="1.1192413e-05" iyz="-1.4400107e-11"
                    izz="2.0712558e-05" />
-      </inertial> -->
+      </inertial>
       <collision name="sg90h_collision">
           <geometry>
@@ -660,6 +594,6 @@
           </geometry>
       </visual> -->
-      </link>
-    <!-- <joint name="sg90h_shaft_joint" type="continuous">
+    </link>
+    <joint name="sg90h_shaft_joint" type="continuous">
       <parent link="sg90h"/>
       <child link="sg90h_shaft"/>
@@ -685,5 +619,5 @@
         </geometry>
       </visual>
-    </link> -->
+    </link>
     <!-- <joint name="sg90v_joint" type="fixed">
       <parent link="supporto_pitch_servo_2"/>
