Commit message: uncommenting and placing parts

File: models/myroboturdf/myrobot.gazebo.xacro (robot description, xacro)
@@ -47,4 +47,7 @@
   </gazebo>
   <gazebo reference="sg90h_shaft">
+    <material>Gazebo/Red</material>
+  </gazebo>
+  <gazebo reference="sg90v_shaft">
     <material>Gazebo/Red</material>
   </gazebo>
@@ -217,7 +220,7 @@
       </plugin>
   </gazebo>
- <!--  <gazebo>
+  <gazebo>
     <plugin name="ActuatorPlugin_vertical" filename="libactuator_plugin.so">
-        <motor_joint>sg90v_to_shaft</motor_joint>
+        <motor_joint>sg90v_shaft_joint</motor_joint>
         <commandTopicServo>cmd_servo</commandTopicServo>
         <servoTorque>10</servoTorque>
@@ -235,4 +238,4 @@
         <rosDebugLevel>na</rosDebugLevel>
       </plugin>
-  </gazebo>-->
+  </gazebo>
   </robot>

File: models/myroboturdf/myrobot.urdf.xacro (robot description, xacro)
@@ -308,5 +308,5 @@
       <parent link="supporto_pitch_servo_1"/>
       <child link="supporto_pitch_servo_2"/>
-      <origin xyz="0.1 0 0" rpy="0 0 0"/>
+      <origin xyz="0 -0.059 -0.02" rpy="0 0 -1.5707"/>
     </joint>
     <link name='supporto_pitch_servo_2'>
@@ -317,66 +317,44 @@
       </collision>
       <visual name='supporto_pitch_servo_2_visual'>
-      <origin xyz="0 0 0.02" rpy="0 3.1415 0" />
+      <origin xyz="-0.042 0 0.02" rpy="0 3.1415 0" />
         <geometry>
           <mesh filename="package://myrobot/models/myroboturdf/meshes/Supports/supporto_pitch_servo_2.stl" scale="0.001 0.001 0.001"/>
         </geometry>
       </visual>
-      <visual name='supporto_pitch_servo_2_visual'>
+      <!-- <visual name='supporto_pitch_servo_2_visual'>
         <geometry>
           <box size="0.002 0.02 0.035"/>
         </geometry>
-      </visual>
-    </link>
-    <!-- <joint name="supporto_pitch_servo_2_noservo_joint" type="fixed">
+      </visual> -->
+    </link>
+    <joint name="supporto_pitch_servo_2_noservo_joint" type="fixed">
       <parent link="supporto_pitch_servo_1"/>
       <child link="supporto_pitch_servo_2_noservo"/>
-      <origin xyz="0.106 -0.056 0.116" rpy="0 0 1.5707"/>
-    </joint>
-    <gazebo>
+      <origin xyz="0 0.059 -0.02" rpy="0 0 -1.5707"/>
+    </joint>
     <link name='supporto_pitch_servo_2_noservo'>
-      <inertial>
-        <mass>0.1</mass>
-        <origin xyz="0.0 0 0" rpy=" 0 0 0"/>
-        <inertia>
-          <ixx>0.001</ixx> <ixy>0</ixy> <ixz>0</ixz>
-          <iyy>0.001</iyy> <iyz>0</iyz>
-          <izz>0.001</izz>
-        </inertia>
-      </inertial>
       <collision name='supporto_pitch_servo_2_noservo_collision'>
         <geometry>
-          <box>
-            <size>0.0075 0.035 0.002</size>
-          </box>
-        </geometry>
-      </collision>
+          <box size="0.0075 0.035 0.002"/>
+        </geometry>
+      </collision>
+     <!-- <visual name='supporto_pitch_servo_2_noservo_visual'>
+      <origin xyz="0.085 0 0.02" rpy="0 3.1415 0" />
+        <geometry>
+          <mesh filename="package://myrobot/models/myroboturdf/meshes/Supports/supporto_pitch_servo_2_noservo.dae"/>
+            scale="0.001 0.001 0.001"/>
+        </geometry>
+      </visual>-->
       <visual name='supporto_pitch_servo_2_noservo_visual'>
-      <pose>0.082 0 -0.001 0 0 3.1415</pose>
-        <geometry>
-          <mesh><uri>model://myrobot/meshes/Supports/supporto_pitch_servo_2_noservo.dae</uri></mesh>
-        </geometry>
-        <material>
-          <ambient>0 0 0.196 0.490</ambient>
-          <diffuse>0.043 0.043 0.043 1</diffuse>
-          <specular>.027 .027 .459 64</specular>
-          <emissive>0.047 0.035 0.286 1</emissive>
-        </material>
-      </visual>
-      <collision name='vertical2_collision'>
-      <pose>-0.002375 0 0.018 0 0 0 </pose>
-        <geometry>
-          <box>
-            <size>0.002 0.019 0.036</size>
-          </box>
-        </geometry>
-      </collision>
-    </link>
-    </gazebo> -->
-    <!-- <joint name="supp_RS_joint" type="fixed">
+        <geometry>
+          <box size="0.002 0.019 0.036"/>
+        </geometry>
+      </visual>
+    </link>
+    <joint name="supp_RS_joint" type="fixed">
       <parent link="sg90v_shaft"/>
       <child link="supp_RS"/>
-      <origin xyz="0.106 -0.002 0.128" rpy="0.128 0 0 3.1415"/>
-    </joint>
-    <gazebo>
+      <origin xyz="0 0 0" rpy="0 0 0"/>
+    </joint>
     <link name='supp_RS'>
       <collision name='collision'>
@@ -388,33 +366,39 @@
       </collision>
      <visual name='supp_RS_visual'>
-      <pose>0.0 0.054 0.013 1.5707 0 1.5707</pose>
-        <geometry>
-          <mesh><uri>model://myrobot/meshes/Supports/Supp_RS.dae</uri></mesh>
-        </geometry>
-        <material>
-          <ambient>0 0 0.196 0.490</ambient>
-          <diffuse>0.043 0.043 0.043 1</diffuse>
-          <specular>.027 .027 .459 64</specular>
-          <emissive>0.047 0.035 0.286 1</emissive>
-        </material>
+     <origin xyz="0.0 0.054 0.013" rpy="1.5707 0 1.5707"/>
+        <geometry>
+          <mesh filename="package://myrobot/models/myroboturdf/meshes/Supports/Supp_RS.dae"/>
+        </geometry>
+      </visual>
+      <visual name='visuall'>
+        <geometry>
+          <box size="0.016 0.105 0.0035"/>
+        </geometry>
       </visual>
       <collision name='vertical3_collision'>
-      <pose>0 0.05 0.01 0 0 0 </pose>
-        <geometry>
-          <box>
-            <size>0.016 0.0035 0.02</size>
-          </box>
-        </geometry>
-      </collision>
+      <origin xyz="0 0.05 0.01" rpy="0 0 0"/>
+        <geometry>
+          <box size="0.016 0.0035 0.02"/>
+        </geometry>
+      </collision>
+      <visual name='vertical3_visual'>
+      <origin xyz="0 0.05 0.01" rpy="0 0 0"/>
+        <geometry>
+          <box size="0.016 0.0035 0.02"/>
+        </geometry>
+      </visual>
       <collision name='vertical4_collision'>
-      <pose>0 -0.05 0.01 0 0 0 </pose>
-        <geometry>
-          <box>
-            <size>0.016 0.0035 0.02</size>
-          </box>
-        </geometry>
-      </collision>
-    </link>
-    </gazebo> -->
+      <origin xyz="0 -0.05 0.01" rpy="0 0 0"/>
+        <geometry>
+          <box size="0.016 0.0035 0.02"/>
+        </geometry>
+      </collision>
+      <visual name='vertical4_visual'>
+      <origin xyz="0 -0.05 0.01" rpy="0 0 0"/>
+        <geometry>
+          <box size="0.016 0.0035 0.02"/>
+        </geometry>
+      </visual>
+    </link>
     <!-- <joint name="RealSense_joint" type="fixed">
       <parent link="supp_RS"/>
@@ -620,8 +604,8 @@
       </visual>
     </link>
-    <!-- <joint name="sg90v_joint" type="fixed">
+    <joint name="sg90v_joint" type="fixed">
       <parent link="supporto_pitch_servo_2"/>
       <child link="sg90v"/>
-      <origin xyz="0.106 0.06595 0.136" rpy="3.1415 0 0"/>
+      <origin xyz="0.011 0 0" rpy="0 0 1.5707"/>
     </joint>
     <link name="sg90v">
@@ -639,14 +623,19 @@
       </collision>
       <visual name="sg90v_visual">
+          <geometry>
+            <box size=".012 0.022 0.022"/>
+          </geometry>
+      </visual>
+      <!-- <visual name="sg90v_visual">
           <origin xyz="0 -0.011 0" rpy=" 0 0 0"/>
           <geometry>
-            <mesh filename="package://myrobot/models/myroboturdf/meshes/Misc/sg90.dae" scale="0.001 0.001 0.001"/>
-          </geometry>
-      </visual>
+            <mesh filename="package://myrobot/models/myroboturdf/meshes/Misc/sg90.dae"/>
+          </geometry>
+      </visual> -->
       </link>
     <joint name="sg90v_shaft_joint" type="continuous">
       <parent link="sg90v"/>
       <child link="sg90v_shaft"/>
-      <origin xyz="0.106 0.048 0.141" rpy="1.5707 0 0"/>
+      <origin xyz="-0.0 0.015 -0.005" rpy="1.5707 0 0 "/>
       <axis xyz="0 0 1"/>
     </joint>
@@ -673,14 +662,7 @@
       <parent link="cube_base"/>
       <child link="batteria"/>
-      <origin xyz="-0.02 0 0.075" rpy="0 0 0"/>
+      <origin xyz="0 0 -0.015" rpy="0 0 0"/>
     </joint>
     <link name="batteria">
-      <inertial>
-          <origin xyz="0 0 0" />
-          <mass value="2.8498940e-02" />
-          <inertia ixx="1.1175580e-05" ixy="-4.2369783e-11" ixz="-5.9381719e-09"
-                   iyy="1.1192413e-05" iyz="-1.4400107e-11"
-                   izz="2.0712558e-05" />
-      </inertial>
       <collision name="batteria_collision">
           <geometry>
@@ -689,10 +671,14 @@
       </collision>
       <visual name="batteria_visual">
+          <geometry>
+            <box size="0.102 0.035 0.025"/>
+          </geometry>
+      </visual>
+      <!-- <visual name="batteria_visual">
           <origin xyz="0 0 -0.012" rpy=" 0 0 0"/>
           <geometry>
-            <mesh filename="package://myrobot/models/myroboturdf/meshes/Misc/Turnigy_2200mAh_3S_20C_Lipo_Pack.dae" scale="0.001 0.001 0.001"/>
-          </geometry>
-      </visual>
+            <mesh filename="package://myrobot/models/myroboturdf/meshes/Misc/Turnigy_2200mAh_3S_20C_Lipo_Pack.dae"/>
+          </geometry>
+      </visual> -->
       </link>
-       -->
 </robot>

Commit message: all plugins working. Model complete exc 4 meshes

File: models/myroboturdf/myrobot.gazebo.xacro (robot description, xacro)
@@ -53,7 +53,7 @@
   </gazebo>
   <gazebo reference="supporto_pitch_servo_1">
-    <!-- <material>Gazebo/Blue</material> -->
-  </gazebo>
-  <!-- <gazebo reference="RealSense">
+     <material>Gazebo/Blue</material>
+  </gazebo>
+  <gazebo reference="RealSense">
     <sensor name="camera" type="depth">
       <update_rate>20</update_rate>
@@ -70,42 +70,5 @@
         </clip>
       </camera>
-    </sensor>
-  </gazebo>-->
-  <!-- <gazebo reference="rightfront_force_sensor">
-    <sensor name="rf_force_sensor" type="contact">
-      <update_rate>30.0</update_rate>
-      <always_on>true</always_on>
-      <contact>
-        <collision>collision_rightfront_collision</collision>
-      </contact>
-    </sensor>
-  </gazebo>
-  <gazebo reference="leftfront_force_sensor">
-    <sensor name="lf_force_sensor" type="contact">
-      <update_rate>30.0</update_rate>
-      <always_on>true</always_on>
-      <contact>
-        <collision>collision_leftfront_collision</collision>
-      </contact>
-    </sensor>
-  </gazebo> -->
-<!-- <gazebo reference="LightSensor">
-    <sensor name='camera' type='depth'>
-      <camera name='camera'>
-        <horizontal_fov>1.047</horizontal_fov>
-        <image>
-          <width>320</width>
-          <height>240</height>
-        </image>
-        <clip>
-          <near>0.1</near>
-          <far>100</far>
-        </clip>
-      </camera>
-    </sensor>
-  </gazebo> -->
-<!-- PLUGINS -->
-  <!-- <gazebo>
-    <plugin name="camera_plugin" filename="libdepth_camera_plugin.so">
+      <plugin name="camera_plugin" filename="libdepth_camera_plugin.so">
       <baseline>0.2</baseline>
       <alwaysOn>true</alwaysOn>
@@ -131,22 +94,49 @@
       <hackBaseline>0</hackBaseline>
     </plugin>
-  </gazebo> -->
-  <!-- <gazebo>
-    <plugin name="gazebo_right_bumper_controller" filename="libcontact_plugin.so">
-      <alwaysOn>true</alwaysOn>
-      <updateRate>30.0</updateRate>
-      <bumperTopicName>/force/rightfront_sensor</bumperTopicName>
-      <frameName>rightfront_force_sensor</frameName>
-    </plugin>
-  </gazebo>
-  <gazebo>
-    <plugin name="gazebo_left_bumper_controller" filename="libcontact_plugin.so">
-      <alwaysOn>true</alwaysOn>
-      <updateRate>30.0</updateRate>
-      <bumperTopicName>/force/leftfront_sensor</bumperTopicName>
-      <frameName>leftfront_force_sensor</frameName>
-    </plugin>
-  </gazebo> -->
-  <!-- <gazebo>
+    </sensor>
+  </gazebo>
+  <gazebo reference="rightfront_force_sensor">
+    <sensor name="rf_force_sensor" type="contact">
+      <update_rate>30.0</update_rate>
+      <always_on>true</always_on>
+      <contact>
+        <collision>collision_rightfront_collision</collision>
+      </contact>
+      <plugin name="gazebo_right_bumper_controller" filename="libcontact_plugin.so">
+        <alwaysOn>true</alwaysOn>
+        <updateRate>30.0</updateRate>
+        <bumperTopicName>/force/rightfront_sensor</bumperTopicName>
+        <frameName>rightfront_force_sensor</frameName>
+      </plugin>
+    </sensor>
+  </gazebo>
+  <gazebo reference="leftfront_force_sensor">
+    <sensor name="lf_force_sensor" type="contact">
+      <update_rate>30.0</update_rate>
+      <always_on>true</always_on>
+      <contact>
+        <collision>collision_leftfront_collision</collision>
+      </contact>
+      <plugin name="gazebo_left_bumper_controller" filename="libcontact_plugin.so">
+        <alwaysOn>true</alwaysOn>
+        <updateRate>30.0</updateRate>
+        <bumperTopicName>/force/leftfront_sensor</bumperTopicName>
+        <frameName>leftfront_force_sensor</frameName>
+      </plugin>
+    </sensor>
+  </gazebo>
+<gazebo reference="LightSensor">
+    <sensor name='camera' type='depth'>
+      <camera name='camera'>
+        <horizontal_fov>1.047</horizontal_fov>
+        <image>
+          <width>320</width>
+          <height>240</height>
+        </image>
+        <clip>
+          <near>0.1</near>
+          <far>100</far>
+        </clip>
+      </camera>
     <plugin name="light_sensor_plugin" filename="liblight_sensor_plugin.so">
       <cameraName>camera2</cameraName>
@@ -169,10 +159,11 @@
       <robotNamespace>base_footprint</robotNamespace>
     </plugin>
-  </gazebo> -->
+    </sensor>
+  </gazebo>
   <gazebo reference="laser_sensor">
     <sensor type="ray" name="lds_lfcd_sensor">
       <pose>0 0 0 0 0 0</pose>
-      <visualize>false</visualize>
-      <update_rate>5</update_rate>
+      <visualize>true</visualize>
+      <update_rate>10</update_rate>
       <ray>
         <scan>

File: models/myroboturdf/myrobot.urdf.xacro (robot description, xacro)
@@ -146,4 +146,5 @@
           <mesh filename="package://myrobot/models/myroboturdf/meshes/Supports/BaseBoards.STL" scale="0.001 0.001 0.001"/>
         </geometry>
+        <material name="blue"/>
       </visual>
        <!-- <visual name="BaseBoards_visual">
@@ -164,4 +165,5 @@
           <cylinder length="0.04" radius="0.002"/>
         </geometry>
+        <material name="grey"/>
       </visual>
       <collision name = "stick2_collision">
@@ -176,4 +178,5 @@
           <cylinder length="0.04" radius="0.002"/>
         </geometry>
+        <material name="grey"/>
       </visual>
       <collision name = "stick3_collision">
@@ -188,4 +191,5 @@
           <cylinder length="0.04" radius="0.002"/>
         </geometry>
+        <material name="grey"/>
       </visual>
       <collision name = "stick4_collision">
@@ -200,4 +204,5 @@
           <cylinder length="0.04" radius="0.002"/>
         </geometry>
+        <material name="grey"/>
       </visual>
     </link>
@@ -214,10 +219,10 @@
         </geometry>
       </collision>
-      <visual name ="piastra_anteriore_visual">
+      <!-- <visual name ="piastra_anteriore_visual">
         <origin xyz="0 0 0 " rpy="0 0 0"/>
         <geometry>
           <box size="0.086 0.079320 0.003"/>
         </geometry>
-      </visual>
+      </visual> -->
       <visual>
         <origin xyz="0.025 0 -0.0015 " rpy="0 0 1.5707"/>
@@ -225,4 +230,5 @@
           <mesh filename="package://myrobot/models/myroboturdf/meshes/Supports/Piastra_anteriore2.stl" scale="0.001 0.001 0.001"/>
         </geometry>
+        <material name="grey"/>
       </visual>
     </link>
@@ -258,9 +264,4 @@
     </joint>
     <link name="supporto_piastra_albero">
-      <inertial>
-        <mass value="0.2"/>
-        <origin rpy="0.078 -0.004 0.104" xyz="0 0 0"/>
-        <inertia ixx="0.00052666666" ixy="0" ixz="0" iyy="0.00052666666" iyz="0" izz="0.001"/>
-      </inertial>
       <collision name="supporto_piastra_albero_collision">
         <origin xyz="0 0 0 " rpy="0 0 0"/>
@@ -269,10 +270,10 @@
         </geometry>
       </collision>
-      <visual name="supporto_piastra_albero_visual">
+      <!-- <visual name="supporto_piastra_albero_visual">
         <origin xyz="0 0 0 " rpy="0 0 0"/>
         <geometry>
           <cylinder length="0.004" radius="0.008"/>
         </geometry>
-      </visual>
+      </visual> -->
       <visual name="supporto_piastra_albero_visual">
         <origin xyz="0 0 -0.002" rpy="1.5707 0 4.71238"/>
@@ -297,5 +298,5 @@
           <box size="0.035 0.12 0.003"/>
         </geometry>
-      </visual> -->
+      </visual>  -->
       <visual name='supporto_pitch_servo_1_visual'>
       <origin xyz="0 0 0.004" rpy="3.1415 0 1.5707" />
@@ -326,6 +327,6 @@
           <box size="0.002 0.02 0.035"/>
         </geometry>
-      </visual> -->
-    </link>
+      </visual>  -->
+    </link>-->
     <joint name="supporto_pitch_servo_2_noservo_joint" type="fixed">
       <parent link="supporto_pitch_servo_1"/>
@@ -339,5 +340,5 @@
         </geometry>
       </collision>
-     <!-- <visual name='supporto_pitch_servo_2_noservo_visual'>
+      <!-- <visual name='supporto_pitch_servo_2_noservo_visual'>
       <origin xyz="0.085 0 0.02" rpy="0 3.1415 0" />
         <geometry>
@@ -345,5 +346,5 @@
             scale="0.001 0.001 0.001"/>
         </geometry>
-      </visual>-->
+      </visual> -->
       <visual name='supporto_pitch_servo_2_noservo_visual'>
         <geometry>
@@ -355,20 +356,18 @@
       <parent link="sg90v_shaft"/>
       <child link="supp_RS"/>
-      <origin xyz="0 0 0" rpy="0 0 0"/>
+      <origin xyz="0 0.010 -0.055" rpy="1.5707 0 0"/>
     </joint>
     <link name='supp_RS'>
       <collision name='collision'>
         <geometry>
-          <box>
-            <size>0.016 0.105 0.0035</size>
-          </box>
-        </geometry>
-      </collision>
-     <visual name='supp_RS_visual'>
+          <box size="0.016 0.105 0.0035"/>
+        </geometry>
+      </collision>
+      <!-- <visual name='supp_RS_visual'>
      <origin xyz="0.0 0.054 0.013" rpy="1.5707 0 1.5707"/>
         <geometry>
           <mesh filename="package://myrobot/models/myroboturdf/meshes/Supports/Supp_RS.dae"/>
         </geometry>
-      </visual>
+      </visual>  -->
       <visual name='visuall'>
         <geometry>
@@ -401,10 +400,17 @@
       </visual>
     </link>
-    <!-- <joint name="RealSense_joint" type="fixed">
+    <joint name="RealSense_joint" type="fixed">
       <parent link="supp_RS"/>
       <child link="RealSense"/>
-      <origin xyz="0.108 -0.0075 0.14" rpy="0 0 0"/>
+      <origin xyz="0 0 0.013" rpy="0 0 0"/>
     </joint>
     <link name="RealSense">
+        <inertial>
+          <origin xyz="0 0 0" />
+          <mass value="2.8498940e-02" />
+          <inertia ixx="1.1175580e-05" ixy="-4.2369783e-11" ixz="-5.9381719e-09"
+                   iyy="1.1192413e-05" iyz="-1.4400107e-11"
+                   izz="2.0712558e-05" />
+        </inertial>
         <collision name="RealSense_collision">
           <geometry>
@@ -412,11 +418,18 @@
           </geometry>
         </collision>
-        <visual name="RealSense_visual">
+        <visual name="RealSense_visual2">
+          <geometry>
+            <box size="0.025 0.087 0.02"/>
+          </geometry>
+          <material name="white"/>
+        </visual>
+        <!-- <visual name="RealSense_visual">
           <origin xyz="0.0125 0.0 0" rpy="1.5707 0 1.5707"/>
           <geometry>
-            <mesh filename="package:///myrobot/models/myroboturdf/meshes/Sensors/IntelRealsense_D435_Multibody.dae" scale="1 1 1"/>
-          </geometry>
-        </visual>
-    </link> -->
+            <mesh filename="package://myrobot/models/myroboturdf/meshes/Sensors/IntelRealsense_D435_Multibody.dae"/>
+          </geometry>
+          <material name="white"/>
+        </visual> -->
+    </link>
     <joint name="rightfront_force_sensor_joint" type="fixed">
       <parent link="cube_base"/>
@@ -487,5 +500,5 @@
       <parent link="cube_base"/>
       <child link="laser_sensor"/>
-      <origin xyz="0 0 0 " rpy="0 0 0"/>
+      <origin xyz="0 0 0.15 " rpy="0 0 0"/>
     </joint>
     <link name="laser_sensor">
@@ -627,10 +640,10 @@
           </geometry>
       </visual>
-      <!-- <visual name="sg90v_visual">
+       <!-- <visual name="sg90v_visual">
           <origin xyz="0 -0.011 0" rpy=" 0 0 0"/>
           <geometry>
             <mesh filename="package://myrobot/models/myroboturdf/meshes/Misc/sg90.dae"/>
           </geometry>
-      </visual> -->
+      </visual>  -->
       </link>
     <joint name="sg90v_shaft_joint" type="continuous">

Commit message: map not showing

File: models/myroboturdf/myrobot.gazebo.xacro (robot description, xacro)
@@ -192,5 +192,5 @@
     </sensor>
   </gazebo>
-  <gazebo>
+    <!-- <gazebo>
      <plugin name="ActuatorPlugin_horizontal" filename="libactuator_plugin.so">
         <motor_joint>sg90h_shaft_joint</motor_joint>
@@ -229,4 +229,4 @@
         <rosDebugLevel>na</rosDebugLevel>
       </plugin>
-  </gazebo>
+  </gazebo> -->
   </robot>

File: models/myroboturdf/myrobot.urdf.xacro (robot description, xacro)
@@ -592,5 +592,5 @@
       </visual> -->
     </link>
-    <joint name="sg90h_shaft_joint" type="continuous">
+    <joint name="sg90h_shaft_joint" type="fixed">
       <parent link="sg90h"/>
       <child link="sg90h_shaft"/>
@@ -600,5 +600,5 @@
     <link name="sg90h_shaft">
       <inertial>
-          <origin xyz="0 0 0" />
+          <origin rpy="0 0 0" xyz="0 0 0"/>
           <mass value="2.8498940e-02" />
           <inertia ixx="1.1175580e-05" ixy="-4.2369783e-11" ixz="-5.9381719e-09"
@@ -624,5 +624,5 @@
     <link name="sg90v">
       <inertial>
-          <origin xyz="0 0 0" />
+          <origin rpy="0 0 0" xyz="0 0 0"/>
           <mass value="2.8498940e-02" />
           <inertia ixx="1.1175580e-05" ixy="-4.2369783e-11" ixz="-5.9381719e-09"
@@ -647,5 +647,5 @@
       </visual>  -->
       </link>
-    <joint name="sg90v_shaft_joint" type="continuous">
+    <joint name="sg90v_shaft_joint" type="fixed">
       <parent link="sg90v"/>
       <child link="sg90v_shaft"/>
