Commit message: robot moves flawlessly

File: models/myroboturdf/myrobot.gazebo.xacro (robot description, xacro)
@@ -10,7 +10,7 @@
     <kd>10.0</kd>
     <minDepth>0.001</minDepth>
-    <maxVel>1</maxVel>
+    <maxVel>0.1</maxVel>
     <fdir1>1 0 0</fdir1>
-    <material>light_black</material>
+    <material>Gazebo/FlatBlack</material>
   </gazebo>
   <gazebo reference="wheel_right_link">
@@ -20,8 +20,17 @@
     <kd>10.0</kd>
     <minDepth>0.001</minDepth>
-    <maxVel>1</maxVel>
+    <maxVel>0.1</maxVel>
     <fdir1>1 0 0</fdir1>
     <material>Gazebo/FlatBlack</material>
   </gazebo>
+  <!-- <gazebo reference="caster_back_link">
+    <mu1>0.1</mu1>
+    <mu2>0.1</mu2>
+    <kp>1000000.0</kp>
+    <kd>100.0</kd>
+    <minDepth>0.001</minDepth>
+    <maxVel>1.0</maxVel>
+    <material>Gazebo/FlatBlack</material>
+  </gazebo> -->
    <gazebo>
     <plugin name="turtlebot3_burger_controller" filename="libdiff_drive_plugin.so">
@@ -46,14 +55,14 @@
     </plugin>
   </gazebo>
-  <gazebo reference="sg90h_shaft">
+  <!-- <gazebo reference="sg90h_shaft">
     <material>Gazebo/Red</material>
   </gazebo>
   <gazebo reference="sg90v_shaft">
     <material>Gazebo/Red</material>
-  </gazebo>
-  <gazebo reference="supporto_pitch_servo_1">
+  </gazebo> -->
+  <!-- <gazebo reference="supporto_pitch_servo_1">
      <material>Gazebo/Blue</material>
-  </gazebo>
-  <gazebo reference="RealSense">
+  </gazebo> -->
+  <!-- <gazebo reference="RealSense">
     <sensor name="camera" type="depth">
       <update_rate>20</update_rate>
@@ -95,6 +104,6 @@
     </plugin>
     </sensor>
-  </gazebo>
-  <gazebo reference="rightfront_force_sensor">
+  </gazebo> -->
+  <!-- <gazebo reference="rightfront_force_sensor">
     <sensor name="rf_force_sensor" type="contact">
       <update_rate>30.0</update_rate>
@@ -125,6 +134,6 @@
       </plugin>
     </sensor>
-  </gazebo>
-<gazebo reference="LightSensor">
+  </gazebo> -->
+<!-- <gazebo reference="LightSensor">
     <sensor name='camera' type='depth'>
       <camera name='camera'>
@@ -160,9 +169,9 @@
     </plugin>
     </sensor>
-  </gazebo>
-  <gazebo reference="laser_sensor">
+  </gazebo> -->
+  <!-- <gazebo reference="laser_sensor">
     <sensor type="ray" name="lds_lfcd_sensor">
       <pose>0 0 0 0 0 0</pose>
-      <visualize>true</visualize>
+      <visualize>false</visualize>
       <update_rate>10</update_rate>
       <ray>
@@ -191,5 +200,5 @@
       </plugin>
     </sensor>
-  </gazebo>
+  </gazebo> -->
     <!-- <gazebo>
      <plugin name="ActuatorPlugin_horizontal" filename="libactuator_plugin.so">

File: models/myroboturdf/myrobot.urdf.xacro (robot description, xacro)
@@ -13,9 +13,14 @@
       <inertial>
         <origin xyz="0 0 0" rpy="0 0 0"/>
-        <mass value="0.2"/>
+        <mass value="8.2573504e-01"/>
         <inertia ixx="2.2124416e-03" ixy="-1.2294101e-05" ixz="3.4938785e-05"
                  iyy="2.1193702e-03" iyz="-5.0120904e-06"
                  izz="2.0064271e-03" />
       </inertial>
+      <!-- <inertial>
+        <mass value="1.5"/>
+        <origin xyz="0 0 0"/>
+        <inertia ixx="1000" ixy="0" ixz="0" iyy="1000" iyz="0" izz="0.0653"/>
+      </inertial> -->
       <collision name="cube_base_collision">
         <origin xyz="0 0 0 " rpy="0 0 0"/>
@@ -24,16 +29,16 @@
         </geometry>
       </collision>
-     <!-- <visual name="cube_base_visual">
+     <visual name="cube_base_visual">
         <geometry>
           <box size="0.19 0.134 0.047"/>
         </geometry>
-      </visual> -->
-      <visual name="cube_base_visual">
+      </visual>
+      <!-- <visual name="cube_base_visual">
         <origin xyz="0.02 0 -0.01" rpy="1.5707 0 1.5707"/>
         <geometry>
           <mesh filename="package://myrobot/models/myroboturdf/meshes/Devastator.stl" scale="0.001 0.001 0.001"/>
         </geometry>
-        <material name="light_black"/> <!--rviz colour-->
-      </visual>
+        <material name="light_black"/>
+      </visual> -->
       <collision name = "caster_collision">
       <origin xyz="-0.05 0 -0.03" rpy="0 0 0"/>
@@ -52,10 +57,10 @@
         </surface>
       </collision>
-      <!-- <visual name="caster_visual">
+      <visual name="caster_visual">
       <origin xyz="-0.05 0 -0.03" rpy="0 0 0"/>
         <geometry>
           <sphere radius="0.05"/>
         </geometry>
-      </visual> -->
+      </visual>
       <collision name = 'caster2_collision'>
       <origin xyz="0.05 0 -0.03" rpy="0 0 0"/>
@@ -74,15 +79,41 @@
         </surface>
       </collision>
-     <!-- <visual name="caster2_visual">
+     <visual name="caster2_visual">
       <origin xyz="0.05 0 -0.03" rpy="0 0 0"/>
         <geometry>
           <sphere radius="0.05"/>
         </geometry>
-      </visual> -->
-    </link>
+      </visual>
+    </link>
+<!--
+  <joint name="caster_back_joint" type="fixed">
+    <parent link="cube_base"/>
+    <child link="caster_back_link"/>
+    <origin xyz="0.07 0 -0.03" rpy="0 0 0"/>
+  </joint>
+  <link name="caster_back_link">
+    <collision>
+      <origin xyz="0 0 0" rpy="0 0 0"/>
+      <geometry>
+          <sphere radius="0.05"/>
+        </geometry>
+    </collision>
+    <inertial>
+      <origin xyz="0 0 0" />
+      <mass value="0.005" />
+      <inertia ixx="0.001" ixy="0.0" ixz="0.0"
+               iyy="0.001" iyz="0.0"
+               izz="0.001" />
+    </inertial>
+    <visual>
+      <geometry>
+          <sphere radius="0.05"/>
+        </geometry>
+    </visual>
+  </link> -->
     <joint name="wheel_left_joint" type="continuous">
       <parent link="cube_base"/>
       <child link="wheel_left_link"/>
-      <origin xyz="0. 0.087 -0.021" rpy="-1.57 0 0"/>
+      <origin xyz="-0.0 0.087 -0.013" rpy="-1.57 0 0"/>
       <axis xyz="0 0 1"/>
     </joint>
@@ -95,18 +126,18 @@
       <collision name="wheel_left_link_collision">
         <geometry>
-          <cylinder length="0.035" radius="0.06"/>
-        </geometry>
-      </collision>
-      <!-- <visual name="wheel_left_link_visual">
+          <cylinder length="0.035" radius="0.06825"/>
+        </geometry>
+      </collision>
+      <visual name="wheel_left_link_visual">
         <origin xyz="0 0 0" rpy="0 0 0"/>
         <geometry>
-          <cylinder length="0.035" radius="0.06"/>
-        </geometry>
-      </visual> -->
+          <cylinder length="0.035" radius="0.06825"/>
+        </geometry>
+      </visual>
     </link>
     <joint name="wheel_right_joint" type="continuous">
       <parent link="cube_base"/>
       <child link="wheel_right_link"/>
-      <origin xyz="0. -0.087 -0.021" rpy="-1.57 0 0"/>
+      <origin xyz="-0.0 -0.087 -0.013" rpy="-1.57 0 0"/>
       <axis xyz="0 0 1"/>
     </joint>
@@ -119,13 +150,13 @@
       <collision name="wheel_right_link_collision">
         <geometry>
-          <cylinder length="0.035" radius="0.06"/>
-        </geometry>
-      </collision>
-      <!-- <visual name="wheel_right_link_visual">
+          <cylinder length="0.035" radius="0.06825"/>
+        </geometry>
+      </collision>
+      <visual name="wheel_right_link_visual">
         <origin xyz="0 0 0" rpy="0 0 0"/>
         <geometry>
-          <cylinder length="0.035" radius="0.06"/>
-        </geometry>
-      </visual> -->
+          <cylinder length="0.035" radius="0.06825"/>
+        </geometry>
+      </visual>
     </link>
     <joint name="BaseBoards_joint" type="fixed">
@@ -141,5 +172,5 @@
         </geometry>
       </collision>
-      <visual  name="BaseBoards_visual">
+      <!-- <visual  name="BaseBoards_visual">
         <origin xyz="0.05 0 0" rpy="0 0 1.5707"/>
         <geometry>
@@ -147,11 +178,11 @@
         </geometry>
         <material name="blue"/>
-      </visual>
-       <!-- <visual name="BaseBoards_visual">
+      </visual> -->
+       <visual name="BaseBoards_visual">
         <origin xyz="0 0 0" rpy="0 0 0"/>
         <geometry>
           <box size="0.16 0.122315 0.002"/>
         </geometry>
-      </visual> -->
+      </visual>
       <collision name = "stick1_collision">
       <origin xyz="0.075 0.05 -0.02 " rpy="0 0 0"/>
@@ -219,11 +250,11 @@
         </geometry>
       </collision>
-      <!-- <visual name ="piastra_anteriore_visual">
+      <visual name ="piastra_anteriore_visual">
         <origin xyz="0 0 0 " rpy="0 0 0"/>
         <geometry>
           <box size="0.086 0.079320 0.003"/>
         </geometry>
-      </visual> -->
-      <visual>
+      </visual>
+      <!-- <visual>
         <origin xyz="0.025 0 -0.0015 " rpy="0 0 1.5707"/>
         <geometry>
@@ -231,5 +262,5 @@
         </geometry>
         <material name="grey"/>
-      </visual>
+      </visual> -->
     </link>
     <joint name="supporto_sg90_joint" type="fixed">
@@ -245,16 +276,16 @@
         </geometry>
       </collision>
-      <visual>
+      <!-- <visual>
         <origin xyz="-0.003 0.015 0" rpy="0 0 1.5707"/>
         <geometry>
           <mesh filename="package://myrobot/models/myroboturdf/meshes/Supports/Supporto_sg90_base.stl" scale="0.001 0.001 0.001"/>
         </geometry>
-      </visual>
-      <!-- <visual name="supporto_sg90_visual">
+      </visual> -->
+      <visual name="supporto_sg90_visual">
         <origin xyz="0 0 0 " rpy="0 0 0"/>
         <geometry>
           <box size="0.027 0.049 0.004"/>
         </geometry>
-      </visual> -->
+      </visual>
     </link>
     <joint name="supporto_piastra_albero_joint" type="fixed">
@@ -270,16 +301,16 @@
         </geometry>
       </collision>
+      <visual name="supporto_piastra_albero_visual">
+        <origin xyz="0 0 0 " rpy="0 0 0"/>
+        <geometry>
+          <cylinder length="0.004" radius="0.008"/>
+        </geometry>
+      </visual>
       <!-- <visual name="supporto_piastra_albero_visual">
-        <origin xyz="0 0 0 " rpy="0 0 0"/>
-        <geometry>
-          <cylinder length="0.004" radius="0.008"/>
-        </geometry>
-      </visual> -->
-      <visual name="supporto_piastra_albero_visual">
         <origin xyz="0 0 -0.002" rpy="1.5707 0 4.71238"/>
         <geometry>
           <mesh filename="package://myrobot/models/myroboturdf/meshes/Supports/Supporto_piastra_albero.stl" scale="0.001 0.001 0.001"/>
         </geometry>
-      </visual>
+      </visual>  -->
     </link>
     <joint name="supporto_pitch_servo_1_joint" type="fixed">
@@ -294,15 +325,15 @@
         </geometry>
       </collision>
-      <!-- <visual name="supporto_pitch_servo_1_visual">
+      <visual name="supporto_pitch_servo_1_visual">
         <geometry>
           <box size="0.035 0.12 0.003"/>
         </geometry>
-      </visual>  -->
-      <visual name='supporto_pitch_servo_1_visual'>
+      </visual>
+      <!-- <visual name='supporto_pitch_servo_1_visual'>
       <origin xyz="0 0 0.004" rpy="3.1415 0 1.5707" />
         <geometry>
           <mesh filename="package://myrobot/models/myroboturdf/meshes/Supports/supporto_pitch_servo_1_new.stl" scale="0.001 0.001 0.001"/>
         </geometry>
-      </visual>
+      </visual> -->
     </link>
     <joint name="supporto_pitch_servo_2_joint" type="fixed">
@@ -317,16 +348,16 @@
         </geometry>
       </collision>
+      <!-- <visual name='supporto_pitch_servo_2_visual'>
+      <origin xyz="-0.042 0 0.02" rpy="0 3.1415 0" />
+        <geometry>
+          <mesh filename="package://myrobot/models/myroboturdf/meshes/Supports/supporto_pitch_servo_2.stl" scale="0.001 0.001 0.001"/>
+        </geometry>
+      </visual> -->
       <visual name='supporto_pitch_servo_2_visual'>
-      <origin xyz="-0.042 0 0.02" rpy="0 3.1415 0" />
-        <geometry>
-          <mesh filename="package://myrobot/models/myroboturdf/meshes/Supports/supporto_pitch_servo_2.stl" scale="0.001 0.001 0.001"/>
-        </geometry>
-      </visual>
-      <!-- <visual name='supporto_pitch_servo_2_visual'>
         <geometry>
           <box size="0.002 0.02 0.035"/>
         </geometry>
-      </visual>  -->
-    </link>-->
+      </visual>
+    </link>
     <joint name="supporto_pitch_servo_2_noservo_joint" type="fixed">
       <parent link="supporto_pitch_servo_1"/>
@@ -406,5 +437,5 @@
     </joint>
     <link name="RealSense">
-        <inertial>
+        <!-- <inertial>
           <origin xyz="0 0 0" />
           <mass value="2.8498940e-02" />
@@ -412,5 +443,5 @@
                    iyy="1.1192413e-05" iyz="-1.4400107e-11"
                    izz="2.0712558e-05" />
-        </inertial>
+        </inertial> -->
         <collision name="RealSense_collision">
           <geometry>
@@ -504,4 +535,69 @@
     <link name="laser_sensor">
         <inertial>
+          <mass value="0.114" />
+          <origin xyz="0 0 0" />
+          <inertia ixx="0.001" ixy="0.0" ixz="0.0"
+                   iyy="0.001" iyz="0.0"
+                   izz="0.001" />
+        </inertial>
+        <collision name="laser_sensor_collision">
+          <geometry>
+            <box size="0.05 0.01 0.01"/>
+          </geometry>
+        </collision>
+    </link>
+    <joint name="LattePanda_joint" type="fixed">
+      <parent link="BaseBoards"/>
+      <child link="LattePanda"/>
+      <origin xyz="-0.012 0.001 0.002" rpy="0 0 0"/>
+    </joint>
+    <link name="LattePanda">
+      <collision name="LattePanda_collision">
+          <geometry>
+            <box size="0.12 0.08 0.01"/>
+          </geometry>
+      </collision>
+      <visual name="LattePanda_visual">
+          <geometry>
+            <box size="0.12 0.08 0.01"/>
+          </geometry>
+      </visual>
+      <!-- <visual name="LattePanda_visual">
+          <origin xyz="0.001 0 0" rpy="1.5707 0 0 "/>
+          <geometry>
+            <mesh filename="package://myrobot/models/myroboturdf/meshes/Boards/LattePanda_delta.dae"/>
+          </geometry>
+      </visual> -->
+      </link>
+    <joint name="K64F_joint" type="fixed">
+      <parent link="BaseBoards"/>
+      <child link="K64F"/>
+      <origin xyz="0 0 -0.0045" rpy="3.1415 0 1.5707"/>
+    </joint>
+    <link name="K64F">
+      <collision name="K64F_collision">
+          <geometry>
+            <box size="0.085 0.055 0.015"/>
+          </geometry>
+      </collision>
+      <visual name="K64F_visual">
+          <geometry>
+            <box size="0.085 0.055 0.015"/>
+          </geometry>
+      </visual>
+      <!-- <visual name="visual">
+          <origin xyz="-0.037 -0.027 -0.007" rpy=" 0 0 0"/>
+          <geometry>
+            <mesh filename="package://myrobot/models/myroboturdf/meshes/Boards/K64F.dae"/>
+          </geometry>
+      </visual> -->
+      </link>
+    <joint name="sg90h_joint" type="fixed">
+      <parent link="supporto_sg90"/>
+      <child link="sg90h"/>
+      <origin xyz="0.003 -0.00 -0.01" rpy="1.5707 0 0"/>
+    </joint>
+    <link name="sg90h">
+      <!-- <inertial>
           <origin xyz="0 0 0" />
           <mass value="2.8498940e-02" />
@@ -509,70 +605,5 @@
                    iyy="1.1192413e-05" iyz="-1.4400107e-11"
                    izz="2.0712558e-05" />
-        </inertial>
-        <collision name="laser_sensor_collision">
-          <geometry>
-            <box size="0.05 0.01 0.01"/>
-          </geometry>
-        </collision>
-    </link>
-    <joint name="LattePanda_joint" type="fixed">
-      <parent link="BaseBoards"/>
-      <child link="LattePanda"/>
-      <origin xyz="-0.012 0.001 0.002" rpy="0 0 0"/>
-    </joint>
-    <link name="LattePanda">
-      <collision name="LattePanda_collision">
-          <geometry>
-            <box size="0.12 0.08 0.01"/>
-          </geometry>
-      </collision>
-      <visual name="LattePanda_visual">
-          <geometry>
-            <box size="0.12 0.08 0.01"/>
-          </geometry>
-      </visual>
-      <!-- <visual name="LattePanda_visual">
-          <origin xyz="0.001 0 0" rpy="1.5707 0 0 "/>
-          <geometry>
-            <mesh filename="package://myrobot/models/myroboturdf/meshes/Boards/LattePanda_delta.dae"/>
-          </geometry>
-      </visual> -->
-      </link>
-    <joint name="K64F_joint" type="fixed">
-      <parent link="BaseBoards"/>
-      <child link="K64F"/>
-      <origin xyz="0 0 -0.0045" rpy="3.1415 0 1.5707"/>
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
Commit message: aaaaa

File: models/myroboturdf/myrobot.gazebo.xacro (robot description, xacro)
@@ -64,5 +64,5 @@
      <material>Gazebo/Blue</material>
   </gazebo> -->
-  <!-- <gazebo reference="RealSense">
+  <gazebo reference="RealSense">
     <sensor name="camera" type="depth">
       <update_rate>20</update_rate>
@@ -104,5 +104,5 @@
     </plugin>
     </sensor>
-  </gazebo> -->
+  </gazebo>
   <!-- <gazebo reference="rightfront_force_sensor">
     <sensor name="rf_force_sensor" type="contact">
@@ -170,8 +170,8 @@
     </sensor>
   </gazebo> -->
-  <!-- <gazebo reference="laser_sensor">
+  <gazebo reference="laser_sensor">
     <sensor type="ray" name="lds_lfcd_sensor">
       <pose>0 0 0 0 0 0</pose>
-      <visualize>false</visualize>
+      <visualize>true</visualize>
       <update_rate>10</update_rate>
       <ray>
@@ -200,5 +200,5 @@
       </plugin>
     </sensor>
-  </gazebo> -->
+  </gazebo>
     <!-- <gazebo>
      <plugin name="ActuatorPlugin_horizontal" filename="libactuator_plugin.so">

File: models/myroboturdf/myrobot.urdf.xacro (robot description, xacro)
@@ -437,11 +437,4 @@
     </joint>
     <link name="RealSense">
-        <!-- <inertial>
-          <origin xyz="0 0 0" />
-          <mass value="2.8498940e-02" />
-          <inertia ixx="1.1175580e-05" ixy="-4.2369783e-11" ixz="-5.9381719e-09"
-                   iyy="1.1192413e-05" iyz="-1.4400107e-11"
-                   izz="2.0712558e-05" />
-        </inertial> -->
         <collision name="RealSense_collision">
           <geometry>

Commit message: start working with machinelearning pkg

File: models/myroboturdf/myrobot.gazebo.xacro (robot description, xacro)
@@ -48,6 +48,6 @@
       <leftJoint>wheel_left_joint</leftJoint>
       <rightJoint>wheel_right_joint</rightJoint>
-      <wheelSeparation>0.160</wheelSeparation>
-      <wheelDiameter>0.066</wheelDiameter>
+      <wheelSeparation>0.174</wheelSeparation>
+      <wheelDiameter>0.1365</wheelDiameter>
       <wheelAcceleration>1</wheelAcceleration>
       <wheelTorque>10</wheelTorque>
@@ -64,4 +64,33 @@
      <material>Gazebo/Blue</material>
   </gazebo> -->
+  <gazebo>
+    <plugin name="imu_plugin" filename="libgazebo_ros_imu.so">
+      <alwaysOn>true</alwaysOn>
+      <bodyName>imu_link</bodyName>
+      <frameName>imu_link</frameName>
+      <topicName>imu</topicName>
+      <serviceName>imu_service</serviceName>
+      <gaussianNoise>0.0</gaussianNoise>
+      <updateRate>200</updateRate>
+      <imu>
+        <noise>
+          <type>gaussian</type>
+          <rate>
+            <mean>0.0</mean>
+            <stddev>2e-4</stddev>
+            <bias_mean>0.0000075</bias_mean>
+            <bias_stddev>0.0000008</bias_stddev>
+          </rate>
+          <accel>
+            <mean>0.0</mean>
+            <stddev>1.7e-2</stddev>
+            <bias_mean>0.1</bias_mean>
+            <bias_stddev>0.001</bias_stddev>
+          </accel>
+        </noise>
+      </imu>
+    </plugin>
+  </gazebo>
+<!--
   <gazebo reference="RealSense">
     <sensor name="camera" type="depth">
@@ -104,5 +133,5 @@
     </plugin>
     </sensor>
-  </gazebo>
+  </gazebo> -->
   <!-- <gazebo reference="rightfront_force_sensor">
     <sensor name="rf_force_sensor" type="contact">
@@ -178,5 +207,5 @@
         <scan>
           <horizontal>
-            <samples>360</samples>
+            <samples>24</samples>
             <resolution>1</resolution>
             <min_angle>0.0</min_angle>

File: models/myroboturdf/myrobot.urdf.xacro (robot description, xacro)
@@ -431,4 +431,10 @@
       </visual>
     </link>
+  <joint name="imu_joint" type="fixed">
+    <parent link="cube_base"/>
+    <child link="imu_link"/>
+    <origin xyz="0 0 0" rpy="0 0 0"/>
+  </joint>
+  <link name="imu_link"/>
     <joint name="RealSense_joint" type="fixed">
       <parent link="supp_RS"/>

Commit message: minimal changes

File: models/myroboturdf/myrobot.gazebo.xacro (robot description, xacro)
@@ -202,5 +202,5 @@
     <sensor type="ray" name="lds_lfcd_sensor">
       <pose>0 0 0 0 0 0</pose>
-      <visualize>true</visualize>
+      <visualize>false</visualize>
       <update_rate>10</update_rate>
       <ray>

File: models/myroboturdf/myrobot.urdf.xacro (robot description, xacro)
@@ -29,10 +29,10 @@
         </geometry>
       </collision>
-     <visual name="cube_base_visual">
+     <!-- <visual name="cube_base_visual">
         <geometry>
           <box size="0.19 0.134 0.047"/>
         </geometry>
-      </visual>
-      <!-- <visual name="cube_base_visual">
+      </visual> -->
+      <visual name="cube_base_visual">
         <origin xyz="0.02 0 -0.01" rpy="1.5707 0 1.5707"/>
         <geometry>
@@ -40,5 +40,5 @@
         </geometry>
         <material name="light_black"/>
-      </visual> -->
+      </visual>
       <collision name = "caster_collision">
       <origin xyz="-0.05 0 -0.03" rpy="0 0 0"/>
@@ -57,10 +57,10 @@
         </surface>
       </collision>
-      <visual name="caster_visual">
+      <!-- <visual name="caster_visual">
       <origin xyz="-0.05 0 -0.03" rpy="0 0 0"/>
         <geometry>
           <sphere radius="0.05"/>
         </geometry>
-      </visual>
+      </visual> -->
       <collision name = 'caster2_collision'>
       <origin xyz="0.05 0 -0.03" rpy="0 0 0"/>
@@ -79,10 +79,10 @@
         </surface>
       </collision>
-     <visual name="caster2_visual">
+     <!-- <visual name="caster2_visual">
       <origin xyz="0.05 0 -0.03" rpy="0 0 0"/>
         <geometry>
           <sphere radius="0.05"/>
         </geometry>
-      </visual>
+      </visual> -->
     </link>
 <!--
@@ -129,10 +129,10 @@
         </geometry>
       </collision>
-      <visual name="wheel_left_link_visual">
+      <!-- <visual name="wheel_left_link_visual">
         <origin xyz="0 0 0" rpy="0 0 0"/>
         <geometry>
           <cylinder length="0.035" radius="0.06825"/>
         </geometry>
-      </visual>
+      </visual> -->
     </link>
     <joint name="wheel_right_joint" type="continuous">
@@ -153,10 +153,10 @@
         </geometry>
       </collision>
-      <visual name="wheel_right_link_visual">
+      <!-- <visual name="wheel_right_link_visual">
         <origin xyz="0 0 0" rpy="0 0 0"/>
         <geometry>
           <cylinder length="0.035" radius="0.06825"/>
         </geometry>
-      </visual>
+      </visual> -->
     </link>
     <joint name="BaseBoards_joint" type="fixed">
