Commit message: working plugin from nilseuropa

File: models/myroboturdf/myrobot.gazebo.xacro (robot description, xacro)
@@ -33,5 +33,5 @@
     <material>Gazebo/FlatBlack</material>
   </gazebo> -->
-   <gazebo>
+  <gazebo>
     <plugin name="turtlebot3_burger_controller" filename="libdiff_drive_plugin.so">
       <commandTopic>cmd_vel</commandTopic>
@@ -267,3 +267,29 @@
       </plugin>
   </gazebo> -->
+  <!-- attached to left wheel and fully working-->
+  <gazebo>
+    <plugin name="pwm_vel_plugin" filename="libcustom_ros_dc_motor.so">
+        <command_topic>/motor/voltage_norm</command_topic>
+        <velocity_topic>/motor/velocity</velocity_topic>
+        <update_rate>100.0</update_rate>
+        <encoder_topic>/motor/encoder</encoder_topic>
+        <current_topic>/motor/current</current_topic>
+        <supply_topic>/motor/supply_voltage</supply_topic>
+        <motor_nominal_voltage>24.0</motor_nominal_voltage>
+        <moment_of_inertia>0.001</moment_of_inertia>
+        <armature_damping_ratio>0.0001</armature_damping_ratio>
+        <electromotive_force_constant>0.03</electromotive_force_constant>
+        <electric_resistance>13.8</electric_resistance>
+        <electric_inductance>0.001</electric_inductance>
+        <velocity_noise>0.0</velocity_noise>
+        <gear_ratio>72.0</gear_ratio>
+        <publish_velocity>true</publish_velocity>
+        <publish_encoder>true</publish_encoder>
+        <publish_current>false</publish_current>
+        <publish_motor_joint_state>true</publish_motor_joint_state>
+        <encoder_ppr>111</encoder_ppr>
+        <motor_wrench_frame>wheel_left_link</motor_wrench_frame>
+        <motor_shaft_joint>wheel_left_joint</motor_shaft_joint>
+      </plugin>
+  </gazebo>
   </robot>

File: models/myroboturdf/myrobot.urdf.xacro (robot description, xacro)
@@ -130,10 +130,10 @@
         </geometry>
       </collision>
-      <!-- <visual name="wheel_left_link_visual">
+      <visual name="wheel_left_link_visual">
         <origin xyz="0 0 0" rpy="0 0 0"/>
         <geometry>
           <cylinder length="0.035" radius="0.06825"/>
         </geometry>
-      </visual> -->
+      </visual>
     </link>
     <joint name="wheel_right_joint" type="continuous">

Commit message: added plugin to both wheels. modified PWM

File: models/myroboturdf/myrobot.gazebo.xacro (robot description, xacro)
@@ -293,3 +293,29 @@
       </plugin>
   </gazebo>
+  <!-- attached to left wheel and fully working-->
+  <gazebo>
+    <plugin name="pwm_vel_plugin" filename="libcustom_ros_dc_motor.so">
+        <command_topic>/motor/voltage_norm</command_topic>
+        <velocity_topic>/motor/velocity</velocity_topic>
+        <update_rate>100.0</update_rate>
+        <encoder_topic>/motor/encoder</encoder_topic>
+        <current_topic>/motor/current</current_topic>
+        <supply_topic>/motor/supply_voltage</supply_topic>
+        <motor_nominal_voltage>24.0</motor_nominal_voltage>
+        <moment_of_inertia>0.001</moment_of_inertia>
+        <armature_damping_ratio>0.0001</armature_damping_ratio>
+        <electromotive_force_constant>0.03</electromotive_force_constant>
+        <electric_resistance>13.8</electric_resistance>
+        <electric_inductance>0.001</electric_inductance>
+        <velocity_noise>0.0</velocity_noise>
+        <gear_ratio>72.0</gear_ratio>
+        <publish_velocity>true</publish_velocity>
+        <publish_encoder>true</publish_encoder>
+        <publish_current>false</publish_current>
+        <publish_motor_joint_state>true</publish_motor_joint_state>
+        <encoder_ppr>111</encoder_ppr>
+        <motor_wrench_frame>wheel_right_link</motor_wrench_frame>
+        <motor_shaft_joint>wheel_right_joint</motor_shaft_joint>
+      </plugin>
+  </gazebo>
   </robot>

File: models/myroboturdf/myrobot.urdf.xacro (robot description, xacro)
@@ -29,10 +29,10 @@
         </geometry>
       </collision>
-     <!-- <visual name="cube_base_visual">
+     <visual name="cube_base_visual">
         <geometry>
           <box size="0.19 0.134 0.047"/>
         </geometry>
-      </visual> -->
-      <visual name="cube_base_visual">
+      </visual>
+      <!-- <visual name="cube_base_visual">
         <origin xyz="0.02 0 -0.01" rpy="1.5707 0 1.5707"/>
         <geometry>
@@ -40,5 +40,5 @@
         </geometry>
         <material name="light_black"/>
-      </visual>
+      </visual> -->
       <collision name = "caster_collision">
       <origin xyz="-0.05 0 -0.03" rpy="0 0 0"/>
@@ -154,10 +154,10 @@
         </geometry>
       </collision>
-      <!--<visual  name="wheel_right_link_visual">
+      <visual  name="wheel_right_link_visual">
         <origin xyz="0 0 0" rpy="0 0 0"/>
         <geometry>
           <cylinder length="0.035" radius="0.06825"/>
         </geometry>
-      </visual>-->
+      </visual>
     </link>
     <joint name="BaseBoards_joint" type="fixed">

Commit message: working on plugin

File: models/myroboturdf/myrobot.gazebo.xacro (robot description, xacro)
@@ -12,5 +12,5 @@
     <maxVel>0.1</maxVel>
     <fdir1>1 0 0</fdir1>
-    <material>Gazebo/FlatBlack</material>
+    <!-- <material>Gazebo/FlatBlack</material> -->
   </gazebo>
   <gazebo reference="wheel_right_link">
@@ -22,5 +22,5 @@
     <maxVel>0.1</maxVel>
     <fdir1>1 0 0</fdir1>
-    <material>Gazebo/FlatBlack</material>
+    <!-- <material>Gazebo/FlatBlack</material> -->
   </gazebo>
   <!-- <gazebo reference="caster_back_link">

File: models/myroboturdf/myrobot.urdf.xacro (robot description, xacro)
@@ -57,5 +57,4 @@
         </surface>
       </collision>
-<!--
       <visual name="caster_visual">
       <origin xyz="-0.05 0 -0.03" rpy="0 0 0"/>
@@ -63,5 +62,5 @@
           <sphere radius="0.05"/>
         </geometry>
-      </visual> -->
+      </visual>
       <collision name = 'caster2_collision'>
       <origin xyz="0.05 0 -0.03" rpy="0 0 0"/>
@@ -80,10 +79,10 @@
         </surface>
       </collision>
-     <!-- <visual name="caster2_visual">
+     <visual name="caster2_visual">
       <origin xyz="0.05 0 -0.03" rpy="0 0 0"/>
         <geometry>
           <sphere radius="0.05"/>
         </geometry>
-      </visual> -->
+      </visual>
     </link>
 <!--
@@ -469,9 +468,9 @@
     </joint>
     <link name="rightfront_force_sensor">
-        <visual name="rightfront_force_sensor_visual">
+        <!-- <visual name="rightfront_force_sensor_visual">
           <geometry>
             <box size="0.05 0.01 0.01"/>
           </geometry>
-        </visual>
+        </visual> -->
         <collision name="rightfront_force_sensor_collision">
           <geometry>
@@ -486,9 +485,9 @@
     </joint>
     <link name="leftfront_force_sensor">
-        <visual name="leftfront_force_sensor_visual">
+        <!-- <visual name="leftfront_force_sensor_visual">
           <geometry>
             <box size="0.05 0.01 0.01"/>
           </geometry>
-        </visual>
+        </visual> -->
         <collision name="leftfront_force_sensor_collision">
           <geometry>

Commit message: Model,controller work fine. New world

File: models/myroboturdf/myrobot.gazebo.xacro (robot description, xacro)
@@ -92,6 +92,5 @@
     </plugin>
   </gazebo>
-<!--
-  <gazebo reference="RealSense">
+  <!-- <gazebo reference="RealSense">
     <sensor name="camera" type="depth">
       <update_rate>20</update_rate>

File: models/myroboturdf/myrobot.urdf.xacro (robot description, xacro)
@@ -29,10 +29,10 @@
         </geometry>
       </collision>
-     <visual name="cube_base_visual">
+     <!-- <visual name="cube_base_visual">
         <geometry>
           <box size="0.19 0.134 0.047"/>
         </geometry>
-      </visual>
-      <!-- <visual name="cube_base_visual">
+      </visual> -->
+      <visual name="cube_base_visual">
         <origin xyz="0.02 0 -0.01" rpy="1.5707 0 1.5707"/>
         <geometry>
@@ -40,7 +40,7 @@
         </geometry>
         <material name="light_black"/>
-      </visual> -->
+      </visual>
       <collision name = "caster_collision">
-      <origin xyz="-0.05 0 -0.03" rpy="0 0 0"/>
+      <origin xyz="-1 0 -0.03" rpy="0 0 0"/>
         <geometry>
           <sphere radius="0.05"/>
@@ -57,12 +57,12 @@
         </surface>
       </collision>
-      <visual name="caster_visual">
-      <origin xyz="-0.05 0 -0.03" rpy="0 0 0"/>
+      <!-- <visual name="caster_visual">
+      <origin xyz="-1 0 -0.03" rpy="0 0 0"/>
         <geometry>
           <sphere radius="0.05"/>
         </geometry>
-      </visual>
+      </visual> -->
       <collision name = 'caster2_collision'>
-      <origin xyz="0.05 0 -0.03" rpy="0 0 0"/>
+      <origin xyz="1 0 -0.03" rpy="0 0 0"/>
         <geometry>
           <sphere radius="0.05"/>
@@ -79,10 +79,10 @@
         </surface>
       </collision>
-     <visual name="caster2_visual">
-      <origin xyz="0.05 0 -0.03" rpy="0 0 0"/>
+     <!-- <visual name="caster2_visual">
+      <origin xyz="1 0 -0.03" rpy="0 0 0"/>
         <geometry>
           <sphere radius="0.05"/>
         </geometry>
-      </visual>
+      </visual> -->
     </link>
 <!--
@@ -129,4 +129,5 @@
         </geometry>
       </collision>
+<!--
       <visual name="wheel_left_link_visual">
         <origin xyz="0 0 0" rpy="0 0 0"/>
@@ -134,5 +135,5 @@
           <cylinder length="0.035" radius="0.06825"/>
         </geometry>
-      </visual>
+      </visual> -->
     </link>
     <joint name="wheel_right_joint" type="continuous">
@@ -153,10 +154,10 @@
         </geometry>
       </collision>
-      <visual  name="wheel_right_link_visual">
+      <!-- <visual  name="wheel_right_link_visual">
         <origin xyz="0 0 0" rpy="0 0 0"/>
         <geometry>
           <cylinder length="0.035" radius="0.06825"/>
         </geometry>
-      </visual>
+      </visual> -->
     </link>
     <joint name="BaseBoards_joint" type="fixed">
